Commit message: stopped robot from falling through floor and hitting itself, turned on gravity, and added a probably useless attempt at writing a xacro file that took in robotiq and ur5, and fixed the filepath for the MoveIt setup assistant so that it wasn't always looking for the wrong file on Kel's computer

File: ur5_robotiq_description/src/urdf/ur5_robotiq_joint_limited.urdf (robot description, URDF)
Before this commit: robot ur5, 17 links, 16 joints
Links:
- added link world
- link robotiq_85_adapter_link: geometry collision box size=0.064 0.064 0.012; visual box size=0.064 0.064 0.012
- link robotiq_85_base_link: geometry collision mesh filename=package://robotiq_c_model_visualization/meshes/robotiq_85_g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; visual mesh filename=package://robotiq_c_model_visualization/meshes/robotiq_85_g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
- link robotiq_85_left_finger_link: geometry collision mesh filename=package://robotiq_c_model_visualization/meshes/robotiq_85_g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; visual mesh filename=package://robotiq_c_model_visualization/meshes/robotiq_85_g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
- link robotiq_85_left_finger_tip_link: geometry collision mesh filename=package://robotiq_c_model_visualization/meshes/robotiq_85_g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; visual mesh filename=package://robotiq_c_model_visualization/meshes/robotiq_85_g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
- link robotiq_85_left_inner_knuckle_link: geometry collision mesh filename=package://robotiq_c_model_visualization/meshes/robotiq_85_g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; visual mesh filename=package://robotiq_c_model_visualization/meshes/robotiq_85_g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
- link robotiq_85_left_knuckle_link: geometry collision mesh filename=package://robotiq_c_model_visualization/meshes/robotiq_85_g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; visual mesh filename=package://robotiq_c_model_visualization/meshes/robotiq_85_g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
- link robotiq_85_right_finger_link: geometry collision mesh filename=package://robotiq_c_model_visualization/meshes/robotiq_85_g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; visual mesh filename=package://robotiq_c_model_visualization/meshes/robotiq_85_g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
- link robotiq_85_right_finger_tip_link: geometry collision mesh filename=package://robotiq_c_model_visualization/meshes/robotiq_85_g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; visual mesh filename=package://robotiq_c_model_visualization/meshes/robotiq_85_g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
- link robotiq_85_right_inner_knuckle_link: geometry collision mesh filename=package://robotiq_c_model_visualization/meshes/robotiq_85_g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; visual mesh filename=package://robotiq_c_model_visualization/meshes/robotiq_85_g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
- link robotiq_85_right_knuckle_link: geometry collision mesh filename=package://robotiq_c_model_visualization/meshes/robotiq_85_g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; visual mesh filename=package://robotiq_c_model_visualization/meshes/robotiq_85_g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
Joints:
- added joint world_joint: type fixed, parent world, child base_link, origin xyz=0.0 0.0 0.0 rpy=0.0 0.0 0.0

Commit message: Jon fixed everything. New controllers.yaml file, removed fake_execution, moveit plugin topics, controller_list private reference in move_group. Code can now use moveit to control simulated arm in ROS without a robotiq gripper.

File: ur5_robotiq_description/src/urdf/ur5_robotiq_joint_limited.urdf (robot description, URDF)
Before this commit: robot ur5, 18 links, 17 joints
Links:
- removed link robotiq_85_adapter_link
- removed link robotiq_85_base_link
- removed link robotiq_85_left_finger_link
- removed link robotiq_85_left_finger_tip_link
- removed link robotiq_85_left_inner_knuckle_link
- removed link robotiq_85_left_knuckle_link
- removed link robotiq_85_right_finger_link
- removed link robotiq_85_right_finger_tip_link
- removed link robotiq_85_right_inner_knuckle_link
- removed link robotiq_85_right_knuckle_link
- added link ee_fixed_link
Joints:
- removed joint robotiq_85_base_joint
- removed joint robotiq_85_left_finger_joint
- removed joint robotiq_85_left_finger_tip_joint
- removed joint robotiq_85_left_inner_knuckle_joint
- removed joint robotiq_85_left_knuckle_joint
- removed joint robotiq_85_right_finger_joint
- removed joint robotiq_85_right_finger_tip_joint
- removed joint robotiq_85_right_inner_knuckle_joint
- removed joint robotiq_85_right_knuckle_joint
- joint ee_fixed_joint: child robotiq_85_adapter_link -> ee_fixed_link
- joint world_joint: origin xyz=0.0 0.0 0.0 rpy=0.0 0.0 0.0 -> xyz=0.0 0.0 1.0 rpy=0.0 0.0 0.0
