Commit message: Robotiq problems solved: collision checking in MoveIt was not disabled for Robotiq joints. UR5 XACRO file now has some parameters that can be configured to alter the simulation: "show_underactuated" includes the outside "finger" links in the Robotiq gripper, and "gravity" controls whether or not the gripper is affected by gravity. We found problems with the gripper when gravity was enabled.

File: ur5_robotiq_description/src/urdf/robotiq.urdf.xacro (robot description, xacro)
@@ -1,5 +1,5 @@
 <?xml version="1.0" ?>
 <robot name="ur5" xmlns:xacro="http://www.ros.org/wiki/xacro">
-  <xacro:macro name="robotiq_c_model" params="root_link hide_underactuated">
+  <xacro:macro name="robotiq_c_model" params="root_link show_underactuated gravity">
     <joint name="adapter_root_link" type="fixed">
       <parent link="${root_link}" />
@@ -55,5 +55,5 @@
       </collision>
     </link>
-    <xacro:if value="${hide_underactuated}">
+    <xacro:if value="${show_underactuated}">
       <!--  /\  -->
       <!--  /\  -->
@@ -71,5 +71,5 @@
         <origin rpy="1.5707 -1.5707 0" xyz=".04191 -.0306 0"/>
         <limit lower="0" upper="1.5707" velocity="2.0" effort="1000"/>
-        <xacro:if value="${hide_underactuated}">
+        <xacro:if value="${show_underactuated}">
           <mimic joint="robotiq_85_left_knuckle_joint" multiplier="1"/>
         </xacro:if>
@@ -180,5 +180,5 @@
       <origin rpy="1.5707 1.5707 0" xyz=".04843 .0127 0"/>
       <limit lower="0" upper="1.5707" velocity="2.0" effort="1000"/>
-      <xacro:if value="${hide_underactuated}">
+      <xacro:if value="${show_underactuated}">
         <mimic joint="robotiq_85_left_knuckle_joint" offset="0"/>
       </xacro:if>
@@ -190,5 +190,5 @@
       <origin rpy="-1.5707 -1.5707 0" xyz=".04843 -.0127 0"/>
       <limit lower="0" upper="1.5707" velocity="2.0" effort="1000"/>
-      <xacro:if value="${hide_underactuated}">
+      <xacro:if value="${show_underactuated}">
         <mimic joint="robotiq_85_left_knuckle_joint" offset="0"/>
       </xacro:if>
@@ -242,5 +242,5 @@
       <origin rpy="0 0 0" xyz="0 .04196 -.0388"/>
       <limit lower="0" upper="1.5707" velocity="2.0" effort="1000"/>
-      <xacro:if value="${hide_underactuated}">
+      <xacro:if value="${show_underactuated}">
         <mimic joint="robotiq_85_left_knuckle_joint" multiplier="-1"/>
       </xacro:if>
@@ -252,5 +252,5 @@
       <origin rpy="0 0 0" xyz="0 .04196 -.0388"/>
       <limit lower="0" upper="1.5707" velocity="2.0" effort="1000"/>
-      <xacro:if value="${hide_underactuated}">
+      <xacro:if value="${show_underactuated}">
         <mimic joint="robotiq_85_left_knuckle_joint" multiplier="-1"/>
       </xacro:if>
@@ -296,5 +296,5 @@
       </collision>
     </link>
-    <xacro:if value="${hide_underactuated}">
+    <xacro:if value="${show_underactuated}">
       <transmission name="robotiq_85_left_knuckle_trans">
         <type>transmission_interface/SimpleTransmission</type>
@@ -346,56 +346,92 @@
       </actuator>
     </transmission>
-    <gazebo reference="robotiq_85_adapter_link">
-      <selfCollide>true</selfCollide>
-      <gravity>true</gravity>
-      <turnGravityOff>true</turnGravityOff>
-    </gazebo>
-    <gazebo reference="robotiq_85_base_link">
-      <selfCollide>true</selfCollide>
-      <gravity>true</gravity>
-      <turnGravityOff>true</turnGravityOff>
-    </gazebo>
-    <xacro:if value="${hide_underactuated}">
-      <gazebo reference="robotiq_85_left_knuckle_link">
-        <selfCollide>true</selfCollide>
-        <gravity>true</gravity>
-        <turnGravityOff>true</turnGravityOff>
-      </gazebo>
-      <gazebo reference="robotiq_85_right_knuckle_link">
-        <selfCollide>true</selfCollide>
-        <gravity>true</gravity>
-        <turnGravityOff>true</turnGravityOff>
-      </gazebo>
-      <gazebo reference="robotiq_85_left_finger_link">
-        <selfCollide>true</selfCollide>
-        <gravity>true</gravity>
-        <turnGravityOff>true</turnGravityOff>
-      </gazebo>
-      <gazebo reference="robotiq_85_right_finger_link">
-        <selfCollide>true</selfCollide>
-        <gravity>true</gravity>
-        <turnGravityOff>true</turnGravityOff>
+    <xacro:if value="${gravity}">
+      <gazebo reference="robotiq_85_adapter_link">
+        <selfCollide>true</selfCollide>
+        <turnGravityOff>false</turnGravityOff>
+      </gazebo>
+      <gazebo reference="robotiq_85_base_link">
+        <selfCollide>true</selfCollide>
+        <turnGravityOff>false</turnGravityOff>
+      </gazebo>
+      <xacro:if value="${show_underactuated}">
+        <gazebo reference="robotiq_85_left_knuckle_link">
+          <selfCollide>true</selfCollide>
+          <turnGravityOff>false</turnGravityOff>
+        </gazebo>
+        <gazebo reference="robotiq_85_right_knuckle_link">
+          <selfCollide>true</selfCollide>
+          <turnGravityOff>false</turnGravityOff>
+        </gazebo>
+        <gazebo reference="robotiq_85_left_finger_link">
+          <selfCollide>true</selfCollide>
+          <turnGravityOff>false</turnGravityOff>
+        </gazebo>
+        <gazebo reference="robotiq_85_right_finger_link">
+          <selfCollide>true</selfCollide>
+          <turnGravityOff>false</turnGravityOff>
+        </gazebo>
+      </xacro:if>
+      <gazebo reference="robotiq_85_left_inner_knuckle_link">
+        <selfCollide>true</selfCollide>
+        <turnGravityOff>false</turnGravityOff>
+      </gazebo>
+      <gazebo reference="robotiq_85_right_inner_knuckle_link">
+        <selfCollide>true</selfCollide>
+        <turnGravityOff>false</turnGravityOff>
+      </gazebo>
+      <gazebo reference="robotiq_85_left_finger_tip_link">
+        <selfCollide>true</selfCollide>
+        <turnGravityOff>false</turnGravityOff>
+      </gazebo>
+      <gazebo reference="robotiq_85_right_finger_tip_link">
+        <selfCollide>true</selfCollide>
+        <turnGravityOff>false</turnGravityOff>
       </gazebo>
     </xacro:if>
-    <gazebo reference="robotiq_85_left_inner_knuckle_link">
-      <selfCollide>true</selfCollide>
-      <gravity>true</gravity>
-      <turnGravityOff>true</turnGravityOff>
-    </gazebo>
-    <gazebo reference="robotiq_85_right_inner_knuckle_link">
-      <selfCollide>true</selfCollide>
-      <gravity>true</gravity>
-      <turnGravityOff>true</turnGravityOff>
-    </gazebo>
+    <xacro:unless value="${gravity}">
+      <gazebo reference="robotiq_85_adapter_link">
+        <selfCollide>true</selfCollide>
+        <turnGravityOff>true</turnGravityOff>
+      </gazebo>
+      <gazebo reference="robotiq_85_base_link">
+        <selfCollide>true</selfCollide>
+        <turnGravityOff>true</turnGravityOff>
+      </gazebo>
+      <xacro:if value="${show_underactuated}">
+        <gazebo reference="robotiq_85_left_knuckle_link">
+          <selfCollide>true</selfCollide>
+          <turnGravityOff>true</turnGravityOff>
+        </gazebo>
+        <gazebo reference="robotiq_85_right_knuckle_link">
+          <selfCollide>true</selfCollide>
+          <turnGravityOff>true</turnGravityOff>
+        </gazebo>
+        <gazebo reference="robotiq_85_left_finger_link">
+          <selfCollide>true</selfCollide>
+          <turnGravityOff>true</turnGravityOff>
+        </gazebo>
+        <gazebo reference="robotiq_85_right_finger_link">
+          <selfCollide>true</selfCollide>
+          <turnGravityOff>true</turnGravityOff>
+        </gazebo>
+      </xacro:if>
+      <gazebo reference="robotiq_85_left_inner_knuckle_link">
+        <selfCollide>true</selfCollide>
+        <turnGravityOff>true</turnGravityOff>
+      </gazebo>
+      <gazebo reference="robotiq_85_right_inner_knuckle_link">
+        <selfCollide>true</selfCollide>
+        <turnGravityOff>true</turnGravityOff>
+      </gazebo>
+      <gazebo reference="robotiq_85_left_finger_tip_link">
+        <selfCollide>true</selfCollide>
+        <turnGravityOff>true</turnGravityOff>
+      </gazebo>
+      <gazebo reference="robotiq_85_right_finger_tip_link">
+        <selfCollide>true</selfCollide>
+        <turnGravityOff>true</turnGravityOff>
+      </gazebo>
+    </xacro:unless>
   </xacro:macro>
-  <gazebo reference="robotiq_85_left_finger_tip_link">
-    <selfCollide>true</selfCollide>
-    <gravity>true</gravity>
-    <turnGravityOff>true</turnGravityOff>
-  </gazebo>
-  <gazebo reference="robotiq_85_right_finger_tip_link">
-    <selfCollide>true</selfCollide>
-    <gravity>true</gravity>
-    <turnGravityOff>true</turnGravityOff>
-  </gazebo>
 </robot>

File: ur5_robotiq_description/src/urdf/ur5_robotiq_joint_limited.urdf.xacro (robot description, xacro)
@@ -5,6 +5,13 @@
   <xacro:robot></xacro:robot>
   <xacro:include filename="$(find ur5_robotiq_description)/src/urdf/robotiq.urdf.xacro" />
+  <xacro:robotiq_c_model root_link="ee_fixed_link" show_underactuated="false" gravity="false"></xacro:robotiq_c_model>
   <!--
-  <xacro:robotiq_c_model root_link="ee_fixed_link" hide_underactuated="false"></xacro:robotiq_c_model>
+  <xacro:include filename="$(find ur5_robotiq_description)/src/urdf/s_model/s-model_articulated_macro.xacro"/>
+  <xacro:s-model_articulated prefix=""></xacro:s-model_articulated>
+  <joint name="s_model_to_arm" type="fixed">
+    <parent link="ee_fixed_link"/>
+    <child link="palm"/>
+    <origin rpy="0.0 0.0 0.0" xyz="0.0 0.1363 0.0"/>
+  </joint>
   -->
   <!--

Commit message: Gripper now open; weights fixed. Every link in the robotiq gripper used to be 10 kg.

File: ur5_robotiq_description/src/urdf/robotiq.urdf.xacro (robot description, xacro)
@@ -8,5 +8,5 @@
     <link name="robotiq_85_adapter_link">
       <inertial>
-        <mass value="10"/>
+        <mass value="0.1"/>
         <origin xyz="0 0 0" rpy="0 0 0"/>
         <inertia ixx="1" ixy="0" ixz="0" iyy="1" iyz="0" izz="1"/>
@@ -38,5 +38,5 @@
     <link name="robotiq_85_base_link">
       <inertial>
-        <mass value="10"/>
+        <mass value="0.1"/>
         <origin xyz="0 0 0" rpy="0 0 0"/>
         <inertia ixx="1" ixy="0" ixz="0" iyy="1" iyz="0" izz="1"/>
@@ -79,5 +79,5 @@
       <link name="robotiq_85_left_knuckle_link">
         <inertial>
-          <mass value="10"/>
+          <mass value="0.01"/>
           <origin xyz="0 0 0" rpy="0 0 0"/>
           <inertia ixx="1" ixy="0" ixz="0" iyy="1" iyz="0" izz="1"/>
@@ -98,5 +98,5 @@
       <link name="robotiq_85_right_knuckle_link">
         <inertial>
-          <mass value="10"/>
+          <mass value="0.01"/>
           <origin xyz="0 0 0" rpy="0 0 0"/>
           <inertia ixx="1" ixy="0" ixz="0" iyy="1" iyz="0" izz="1"/>
@@ -135,5 +135,5 @@
       <link name="robotiq_85_left_finger_link">
         <inertial>
-          <mass value="10"/>
+          <mass value="0.01"/>
           <origin xyz="0 0 0" rpy="0 0 0"/>
           <inertia ixx="1" ixy="0" ixz="0" iyy="1" iyz="0" izz="1"/>
@@ -154,5 +154,5 @@
       <link name="robotiq_85_right_finger_link">
         <inertial>
-          <mass value="10"/>
+          <mass value="0.01"/>
           <origin xyz="0 0 0" rpy="0 0 0"/>
           <inertia ixx="1" ixy="0" ixz="0" iyy="1" iyz="0" izz="1"/>
@@ -198,5 +198,5 @@
     <link name="robotiq_85_left_inner_knuckle_link">
       <inertial>
-        <mass value="10"/>
+        <mass value="0.01"/>
         <origin xyz="0 0 0" rpy="0 0 0"/>
         <inertia ixx="1" ixy="0" ixz="0" iyy="1" iyz="0" izz="1"/>
@@ -217,5 +217,5 @@
     <link name="robotiq_85_right_inner_knuckle_link">
       <inertial>
-        <mass value="10"/>
+        <mass value="0.01"/>
         <origin xyz="0 0 0" rpy="0 0 0"/>
         <inertia ixx="1" ixy="0" ixz="0" iyy="1" iyz="0" izz="1"/>
@@ -260,5 +260,5 @@
     <link name="robotiq_85_left_finger_tip_link">
       <inertial>
-        <mass value="10"/>
+        <mass value="0.01"/>
         <origin xyz="0 0 0" rpy="0 0 0"/>
         <inertia ixx="1" ixy="0" ixz="0" iyy="1" iyz="0" izz="1"/>
@@ -279,5 +279,5 @@
     <link name="robotiq_85_right_finger_tip_link">
       <inertial>
-        <mass value="10"/>
+        <mass value="0.01"/>
         <origin xyz="0 0 0" rpy="0 0 0"/>
         <inertia ixx="1" ixy="0" ixz="0" iyy="1" iyz="0" izz="1"/>
