Commit message: changes to let us use macros to build UR5's. macro creating the base UR5 as per our previous demos is in base_ur5.urdf.xacro; planning_context now calls the xacro file instead of the urdf.

File: ur5_robotiq_description/src/urdf/base_ur5.urdf.xacro (robot description, xacro)
@@ -1,14 +1,10 @@
 <?xml version="1.0" ?>
 <!-- =================================================================================== -->
-<!-- |    This document was autogenerated by xacro from ur5_robot.urdf.xacro           | -->
+<!-- |    This document was autogenerated by xacro from ur5_joint_limited_robot.urdf.xacro | -->
 <!-- |    EDITING THIS FILE BY HAND IS NOT RECOMMENDED                                 | -->
 <!-- =================================================================================== -->
 <robot name="ur5" xmlns:xacro="http://www.ros.org/wiki/xacro">
   <!-- common stuff -->
-  <gazebo>
-    <plugin filename="libgazebo_ros_controller_manager.so" name="gazebo_ros_controller_manager">
-      <alwaysOn>true</alwaysOn>
-      <updateRate>1000.0</updateRate>
-    </plugin>
+  <!-- <gazebo>
     <plugin filename="libgazebo_ros_power_monitor.so" name="gazebo_ros_power_monitor_controller">
       <alwaysOn>true</alwaysOn>
@@ -22,7 +18,11 @@
       <dischargeVoltage>15.52</dischargeVoltage>
       <chargeVoltage>16.41</chargeVoltage>
+      <selfCollide>true</selfCollide>
+      <turnGravityOff>false</turnGravityOff>
+      <gravity>true</gravity>
     </plugin>
-  </gazebo>
+  </gazebo> -->
   <!-- ur5 -->
+  <xacro:macro name="robot" >
   <material name="UR/Blue">
     <color rgba="0.0 0.0 0.8 1.0"/>
@@ -31,4 +31,10 @@
     <color rgba="0.7 0.7 0.7 1.0"/>
   </material>
+  <link name="world" />
+  <joint name= "world_joint" type="fixed">
+    <parent link="world"/>
+    <child link="base_link"/>
+    <origin rpy="0.0 0.0 0.0" xyz="0.0 0.0 1.0"/>
+  </joint>
   <!-- arm -->
   <link name="base_link">
@@ -55,5 +61,5 @@
     <origin rpy="0.0 0.0 0.0" xyz="0.0 0.0 0.089159"/>
     <axis xyz="0 0 1"/>
-    <limit effort="150.0" lower="-6.2831853" upper="6.2831853" velocity="3.14159265"/>
+    <limit effort="150.0" lower="-3.14159265" upper="3.14159265" velocity="3.14159265"/>
     <dynamics damping="0.4" friction="0.0"/>
   </joint>
@@ -81,5 +87,5 @@
     <origin rpy="0.0 1.570796325 0.0" xyz="0.0 0.13585 0.0"/>
     <axis xyz="0 1 0"/>
-    <limit effort="150.0" lower="-6.2831853" upper="6.2831853" velocity="3.14159265"/>
+    <limit effort="150.0" lower="-3.14159265" upper="3.14159265" velocity="3.14159265"/>
     <dynamics damping="0.4" friction="0.0"/>
   </joint>
@@ -108,5 +114,5 @@
     <origin rpy="0.0 0.0 0.0" xyz="0.0 -0.1197 0.425"/>
     <axis xyz="0 1 0"/>
-    <limit effort="150.0" lower="-6.2831853" upper="6.2831853" velocity="3.14159265"/>
+    <limit effort="150.0" lower="-3.14159265" upper="3.14159265" velocity="3.14159265"/>
     <dynamics damping="0.4" friction="0.0"/>
   </joint>
@@ -262,6 +268,156 @@
     </actuator>
   </transmission>
+  <!-- <transmission name="robotiq_85_left_knuckle_trans">
+    <type>transmission_interface/SimpleTransmission</type>
+    <joint name="robotiq_85_left_knuckle_joint"/>
+    <actuator name="robotiq_85_left_knuckle_motor">
+      <hardwareInterface>PositionJointInterface</hardwareInterface>
+      <mechanicalReduction>1</mechanicalReduction>
+    </actuator>
+  </transmission>
+  <transmission name="robotiq_85_right_knuckle_trans">
+    <type>transmission_interface/SimpleTransmission</type>
+    <joint name="robotiq_85_right_knuckle_joint"/>
+    <actuator name="robotiq_85_right_knuckle_motor">
+      <hardwareInterface>PositionJointInterface</hardwareInterface>
+      <mechanicalReduction>1</mechanicalReduction>
+    </actuator>
+  </transmission>
+  <transmission name="robotiq_85_left_finger_trans">
+    <type>transmission_interface/SimpleTransmission</type>
+    <joint name="robotiq_85_left_finger_joint"/>
+    <actuator name="robotiq_85_left_finger_motor">
+      <hardwareInterface>PositionJointInterface</hardwareInterface>
+      <mechanicalReduction>1</mechanicalReduction>
+    </actuator>
+  </transmission>
+  <transmission name="robotiq_85_right_finger_trans">
+    <type>transmission_interface/SimpleTransmission</type>
+    <joint name="robotiq_85_right_finger_joint"/>
+    <actuator name="robotiq_85_right_finger_motor">
+      <hardwareInterface>PositionJointInterface</hardwareInterface>
+      <mechanicalReduction>1</mechanicalReduction>
+    </actuator>
+  </transmission>
+  <transmission name="robotiq_85_left_inner_knuckle_trans">
+    <type>transmission_interface/SimpleTransmission</type>
+    <joint name="robotiq_85_left_inner_knuckle_joint"/>
+    <actuator name="robotiq_85_left_inner_knuckle_motor">
+      <hardwareInterface>PositionJointInterface</hardwareInterface>
+      <mechanicalReduction>1</mechanicalReduction>
+    </actuator>
+  </transmission>
+  <transmission name="robotiq_85_right_inner_knuckle_trans">
+    <type>transmission_interface/SimpleTransmission</type>
+    <joint name="robotiq_85_right_inner_knuckle_joint"/>
+    <actuator name="robotiq_85_right_inner_knuckle_motor">
+      <hardwareInterface>PositionJointInterface</hardwareInterface>
+      <mechanicalReduction>1</mechanicalReduction>
+    </actuator>
+  </transmission>
+  <transmission name="robotiq_85_left_finger_tip_trans">
+    <type>transmission_interface/SimpleTransmission</type>
+    <joint name="robotiq_85_left_finger_tip_joint"/>
+    <actuator name="robotiq_85_left_finger_tip_motor">
+      <hardwareInterface>PositionJointInterface</hardwareInterface>
+      <mechanicalReduction>1</mechanicalReduction>
+    </actuator>
+  </transmission>
+  <transmission name="robotiq_85_right_finger_tip_trans">
+    <type>transmission_interface/SimpleTransmission</type>
+    <joint name="robotiq_85_right_finger_tip_joint"/>
+    <actuator name="robotiq_85_right_finger_tip_motor">
+      <hardwareInterface>PositionJointInterface</hardwareInterface>
+      <mechanicalReduction>1</mechanicalReduction>
+    </actuator>
+  </transmission> -->
   <gazebo reference="universal_robot">
     <material>Gazebo/Blue</material>
   </gazebo>
+  <gazebo>
+    <plugin name="gazebo_ros_control" filename="libgazebo_ros_control.so">
+      <robotNamespace>/ur5_robotiq_joint_limited</robotNamespace>
+    </plugin>
+  </gazebo>
+  <gazebo reference="base_link">
+      <selfCollide>true</selfCollide>
+      <gravity>true</gravity>
+      <turnGravityOff>false</turnGravityOff>
+  </gazebo>
+  <gazebo reference="upper_arm_link">
+      <selfCollide>true</selfCollide>
+      <gravity>true</gravity>
+      <turnGravityOff>false</turnGravityOff>
+  </gazebo>
+  <gazebo reference="forearm_link">
+      <selfCollide>true</selfCollide>
+      <gravity>true</gravity>
+      <turnGravityOff>false</turnGravityOff>
+  </gazebo>
+  <gazebo reference="wrist_1_link">
+      <selfCollide>true</selfCollide>
+      <gravity>true</gravity>
+      <turnGravityOff>false</turnGravityOff>
+  </gazebo>
+  <gazebo reference="wrist_2_link">
+      <selfCollide>true</selfCollide>
+      <gravity>true</gravity>
+      <turnGravityOff>false</turnGravityOff>
+  </gazebo>
+  <gazebo reference="wrist_3_link">
+      <selfCollide>true</selfCollide>
+      <gravity>true</gravity>
+      <turnGravityOff>false</turnGravityOff>
+  </gazebo>
+  <gazebo reference="robotiq_85_adapter_link">
+      <selfCollide>true</selfCollide>
+      <gravity>true</gravity>
+      <turnGravityOff>false</turnGravityOff>
+  </gazebo>
+  <gazebo reference="robotiq_85_base_link">
+      <selfCollide>true</selfCollide>
+      <gravity>true</gravity>
+      <turnGravityOff>false</turnGravityOff>
+  </gazebo>
+  <gazebo reference="robotiq_85_left_knuckle_link">
+      <selfCollide>true</selfCollide>
+      <gravity>true</gravity>
+      <turnGravityOff>false</turnGravityOff>
+  </gazebo>
+  <gazebo reference="robotiq_85_right_knuckle_link">
+      <selfCollide>true</selfCollide>
+      <gravity>true</gravity>
+      <turnGravityOff>false</turnGravityOff>
+  </gazebo>
+  <gazebo reference="robotiq_85_left_finger_link">
+      <selfCollide>true</selfCollide>
+      <gravity>true</gravity>
+      <turnGravityOff>false</turnGravityOff>
+  </gazebo>
+  <gazebo reference="robotiq_85_right_finger_link">
+      <selfCollide>true</selfCollide>
+      <gravity>true</gravity>
+      <turnGravityOff>false</turnGravityOff>
+  </gazebo>
+  <gazebo reference="robotiq_85_left_inner_knuckle_link">
+      <selfCollide>true</selfCollide>
+      <gravity>true</gravity>
+      <turnGravityOff>false</turnGravityOff>
+  </gazebo>
+  <gazebo reference="robotiq_85_right_inner_knuckle_link">
+      <selfCollide>true</selfCollide>
+      <gravity>true</gravity>
+      <turnGravityOff>false</turnGravityOff>
+  </gazebo>
+    <gazebo reference="robotiq_85_left_finger_tip_link">
+      <selfCollide>true</selfCollide>
+      <gravity>true</gravity>
+      <turnGravityOff>false</turnGravityOff>
+  </gazebo>
+  <gazebo reference="robotiq_85_right_finger_tip_link">
+      <selfCollide>true</selfCollide>
+      <gravity>true</gravity>
+      <turnGravityOff>false</turnGravityOff>
+    </gazebo>
+  </xacro:macro>
 </robot>

File: ur5_robotiq_description/src/urdf/ur5_robotiq_joint_limited.urdf.xacro (robot description, xacro)
@@ -1,26 +1,18 @@
 <?xml version="1.0"?>
 <robot xmlns:xacro="http://www.ros.org/wiki/xacro"
-       name="ur5_robotiq" >
-  <!-- this code has never  been used and should not be used - we just started writing it, but stopped halfway through -->
-  <!-- common stuff -->
+       name="ur5" >
+  <xacro:include filename="$(find ur5_robotiq_description)/src/urdf/base_ur5.urdf.xacro" />
+  <xacro:robot></xacro:robot>
+  <!--
+  <link name="world" />
+  <joint name= "world_joint" type="fixed">
+    <parent link="world"/>
+    <child link="base_link"/>
+    <origin rpy="0.0 0.0 0.0" xyz="0.0 0.0 1.0"/>
+  </joint>
   <xacro:include filename="$(find ur_description)/urdf/gazebo.urdf.xacro" />
-  <!-- ur5 -->
   <xacro:include filename="$(find ur_description)/urdf/ur5_joint_limited.urdf.xacro" />
-  <!-- arm -->
   <xacro:ur5_robot prefix="">
   </xacro:ur5_robot>
-  <!-- robotiq_2_finger -->
-  <xacro:include filename="$(find robotiq)/robotiq_c_model_visualization/models/robotiq_c_model.urdf" />
-  <!-- joint that attaches to connector plate -->
-  <joint name="ee_fixed_joint" type="fixed">
-    <parent link="ee_link"/>
-    <child link="robotiq_85_adapter_link"/>
-    <origin rpy="0.0 0.0 1.570796325" xyz="0.0 0.0823 0.0"/>
-  </joint>
-  <!-- joint to world -->
-  <joint name="world_joint" type="fixed">
-    <parent link="world"/>
-    <child link="robotiq_85_adapter_link"/>
-    <origin rpy="0.0 0.0 1.570796325" xyz="0.0 0.0823 0.0"/>
-  </joint>
+  -->
 </robot>

File: ur_description/urdf/ur5.transmission.xacro (robot description, xacro)
@@ -6,5 +6,5 @@
 			<joint name="${prefix}shoulder_pan_joint"/>
 			<actuator name="${prefix}shoulder_pan_motor">
-				<hardwareInterface>EffortJointInterface</hardwareInterface>
+				<hardwareInterface>PositionJointInterface</hardwareInterface>
 				<mechanicalReduction>1</mechanicalReduction>
 			</actuator>
@@ -14,5 +14,5 @@
 			<joint name="${prefix}shoulder_lift_joint"/>
 			<actuator name="${prefix}shoulder_lift_motor">
-				<hardwareInterface>EffortJointInterface</hardwareInterface>
+				<hardwareInterface>PositionJointInterface</hardwareInterface>
 				<mechanicalReduction>1</mechanicalReduction>
 			</actuator>
@@ -22,5 +22,5 @@
 			<joint name="${prefix}elbow_joint"/>
 			<actuator name="${prefix}elbow_motor">
-				<hardwareInterface>EffortJointInterface</hardwareInterface>
+				<hardwareInterface>PositionJointInterface</hardwareInterface>
 				<mechanicalReduction>1</mechanicalReduction>
 			</actuator>
@@ -30,5 +30,5 @@
 			<joint name="${prefix}wrist_1_joint"/>
 			<actuator name="${prefix}wrist_1_motor">
-				<hardwareInterface>EffortJointInterface</hardwareInterface>
+				<hardwareInterface>PositionJointInterface</hardwareInterface>
 				<mechanicalReduction>1</mechanicalReduction>
 			</actuator>
@@ -38,5 +38,5 @@
 			<joint name="${prefix}wrist_2_joint"/>
 			<actuator name="${prefix}wrist_2_motor">
-				<hardwareInterface>EffortJointInterface</hardwareInterface>
+				<hardwareInterface>PositionJointInterface</hardwareInterface>
 				<mechanicalReduction>1</mechanicalReduction>
 			</actuator>
@@ -46,5 +46,5 @@
 			<joint name="${prefix}wrist_3_joint"/>
 			<actuator name="${prefix}wrist_3_motor">
-				<hardwareInterface>EffortJointInterface</hardwareInterface>
+				<hardwareInterface>PositionJointInterface</hardwareInterface>
 				<mechanicalReduction>1</mechanicalReduction>
 			</actuator>

File: ur_description/urdf/ur5_joint_limited.urdf.xacro (robot description, xacro)
@@ -222,8 +222,8 @@
   <joint name="${prefix}ee_fixed_joint" type="fixed">
     <parent link="${prefix}wrist_3_link" />
-    <child link = "${prefix}ee_link" />
+    <child link = "${prefix}ee_fixed_link" />
     <origin xyz="0.0 ${wrist_3_length} 0.0" rpy="0.0 0.0 ${pi/2.0}" />
   </joint>
-  <link name="${prefix}ee_link" />
+  <link name="${prefix}ee_fixed_link" />
   <xacro:ur5_arm_transmission prefix="${prefix}" />
   <xacro:ur5_arm_gazebo prefix="${prefix}" />
