Commit message: Added option to .xacro file, "hide_underactuated", to hide the outside "fingers" of the Robotiq gripper. Added back in the transmissions for the fingers to the robotiq URDF file, so that they show up correctly in RVIZ and so that MoveIt can plan. MoveIt cannot find valid positions for the gripper, so currently the gripper is disabled in ur5_robotiq_joint_limited.urdf.xacro.

File: ur5_robotiq_description/src/urdf/base_ur5.urdf.xacro (robot description, xacro)
@@ -264,68 +264,4 @@
     </actuator>
   </transmission>
-  <!-- <transmission name="robotiq_85_left_knuckle_trans">
-    <type>transmission_interface/SimpleTransmission</type>
-    <joint name="robotiq_85_left_knuckle_joint"/>
-    <actuator name="robotiq_85_left_knuckle_motor">
-      <hardwareInterface>PositionJointInterface</hardwareInterface>
-      <mechanicalReduction>1</mechanicalReduction>
-    </actuator>
-  </transmission>
-  <transmission name="robotiq_85_right_knuckle_trans">
-    <type>transmission_interface/SimpleTransmission</type>
-    <joint name="robotiq_85_right_knuckle_joint"/>
-    <actuator name="robotiq_85_right_knuckle_motor">
-      <hardwareInterface>PositionJointInterface</hardwareInterface>
-      <mechanicalReduction>1</mechanicalReduction>
-    </actuator>
-  </transmission>
-  <transmission name="robotiq_85_left_finger_trans">
-    <type>transmission_interface/SimpleTransmission</type>
-    <joint name="robotiq_85_left_finger_joint"/>
-    <actuator name="robotiq_85_left_finger_motor">
-      <hardwareInterface>PositionJointInterface</hardwareInterface>
-      <mechanicalReduction>1</mechanicalReduction>
-    </actuator>
-  </transmission>
-  <transmission name="robotiq_85_right_finger_trans">
-    <type>transmission_interface/SimpleTransmission</type>
-    <joint name="robotiq_85_right_finger_joint"/>
-    <actuator name="robotiq_85_right_finger_motor">
-      <hardwareInterface>PositionJointInterface</hardwareInterface>
-      <mechanicalReduction>1</mechanicalReduction>
-    </actuator>
-  </transmission>
-  <transmission name="robotiq_85_left_inner_knuckle_trans">
-    <type>transmission_interface/SimpleTransmission</type>
-    <joint name="robotiq_85_left_inner_knuckle_joint"/>
-    <actuator name="robotiq_85_left_inner_knuckle_motor">
-      <hardwareInterface>PositionJointInterface</hardwareInterface>
-      <mechanicalReduction>1</mechanicalReduction>
-    </actuator>
-  </transmission>
-  <transmission name="robotiq_85_right_inner_knuckle_trans">
-    <type>transmission_interface/SimpleTransmission</type>
-    <joint name="robotiq_85_right_inner_knuckle_joint"/>
-    <actuator name="robotiq_85_right_inner_knuckle_motor">
-      <hardwareInterface>PositionJointInterface</hardwareInterface>
-      <mechanicalReduction>1</mechanicalReduction>
-    </actuator>
-  </transmission>
-  <transmission name="robotiq_85_left_finger_tip_trans">
-    <type>transmission_interface/SimpleTransmission</type>
-    <joint name="robotiq_85_left_finger_tip_joint"/>
-    <actuator name="robotiq_85_left_finger_tip_motor">
-      <hardwareInterface>PositionJointInterface</hardwareInterface>
-      <mechanicalReduction>1</mechanicalReduction>
-    </actuator>
-  </transmission>
-  <transmission name="robotiq_85_right_finger_tip_trans">
-    <type>transmission_interface/SimpleTransmission</type>
-    <joint name="robotiq_85_right_finger_tip_joint"/>
-    <actuator name="robotiq_85_right_finger_tip_motor">
-      <hardwareInterface>PositionJointInterface</hardwareInterface>
-      <mechanicalReduction>1</mechanicalReduction>
-    </actuator>
-  </transmission> -->
   <gazebo reference="universal_robot">
     <material>Gazebo/Blue</material>
@@ -366,54 +302,4 @@
       <turnGravityOff>false</turnGravityOff>
   </gazebo>
-  <gazebo reference="robotiq_85_adapter_link">
-      <selfCollide>true</selfCollide>
-      <gravity>true</gravity>
-      <turnGravityOff>false</turnGravityOff>
-  </gazebo>
-  <gazebo reference="robotiq_85_base_link">
-      <selfCollide>true</selfCollide>
-      <gravity>true</gravity>
-      <turnGravityOff>false</turnGravityOff>
-  </gazebo>
-  <gazebo reference="robotiq_85_left_knuckle_link">
-      <selfCollide>true</selfCollide>
-      <gravity>true</gravity>
-      <turnGravityOff>false</turnGravityOff>
-  </gazebo>
-  <gazebo reference="robotiq_85_right_knuckle_link">
-      <selfCollide>true</selfCollide>
-      <gravity>true</gravity>
-      <turnGravityOff>false</turnGravityOff>
-  </gazebo>
-  <gazebo reference="robotiq_85_left_finger_link">
-      <selfCollide>true</selfCollide>
-      <gravity>true</gravity>
-      <turnGravityOff>false</turnGravityOff>
-  </gazebo>
-  <gazebo reference="robotiq_85_right_finger_link">
-      <selfCollide>true</selfCollide>
-      <gravity>true</gravity>
-      <turnGravityOff>false</turnGravityOff>
-  </gazebo>
-  <gazebo reference="robotiq_85_left_inner_knuckle_link">
-      <selfCollide>true</selfCollide>
-      <gravity>true</gravity>
-      <turnGravityOff>false</turnGravityOff>
-  </gazebo>
-  <gazebo reference="robotiq_85_right_inner_knuckle_link">
-      <selfCollide>true</selfCollide>
-      <gravity>true</gravity>
-      <turnGravityOff>false</turnGravityOff>
-  </gazebo>
-    <gazebo reference="robotiq_85_left_finger_tip_link">
-      <selfCollide>true</selfCollide>
-      <gravity>true</gravity>
-      <turnGravityOff>false</turnGravityOff>
-  </gazebo>
-  <gazebo reference="robotiq_85_right_finger_tip_link">
-      <selfCollide>true</selfCollide>
-      <gravity>true</gravity>
-      <turnGravityOff>false</turnGravityOff>
-    </gazebo>
   </xacro:macro>
 </robot>

File: ur5_robotiq_description/src/urdf/robotiq.urdf.xacro (robot description, xacro)
@@ -1,5 +1,5 @@
 <?xml version="1.0" ?>
 <robot name="ur5" xmlns:xacro="http://www.ros.org/wiki/xacro">
-  <xacro:macro name="robotiq_c_model" params="root_link">
+  <xacro:macro name="robotiq_c_model" params="root_link hide_underactuated">
     <joint name="adapter_root_link" type="fixed">
       <parent link="${root_link}" />
@@ -55,117 +55,121 @@
       </collision>
     </link>
-    <!--  /\  -->
-    <!--  /\  -->
-    <joint name="robotiq_85_left_knuckle_joint" type="revolute">
-      <parent link="robotiq_85_base_link"/>
-      <child link="robotiq_85_left_knuckle_link"/>
-      <axis xyz="1 0 0"/>
-      <origin rpy="-1.5707 1.5707 0" xyz=".04191 .0306 0"/>
-      <limit lower="0" upper=".8575" velocity="2.0" effort="1000"/>
-    </joint>
-    <joint name="robotiq_85_right_knuckle_joint" type="revolute">
-      <parent link="robotiq_85_base_link"/>
-      <child link="robotiq_85_right_knuckle_link"/>
-      <axis xyz="1 0 0"/>
-      <origin rpy="1.5707 -1.5707 0" xyz=".04191 -.0306 0"/>
-      <limit lower="0" upper="1.5707" velocity="2.0" effort="1000"/>
-      <mimic joint="robotiq_85_left_knuckle_joint" multiplier="1"/>
-    </joint>
-    <!--  \/  -->
-    <!--  \/  -->
-    <link name="robotiq_85_left_knuckle_link">
-      <inertial>
-        <mass value="10"/>
-        <origin xyz="0 0 0" rpy="0 0 0"/>
-        <inertia ixx="1" ixy="0" ixz="0" iyy="1" iyz="0" izz="1"/>
-      </inertial>
-      <visual>
-        <geometry>
-          <mesh filename="package://robotiq_c_model_visualization/meshes/robotiq_85_gripper_joint_0_L.dae"/>
-        </geometry>
-        <origin rpy="3.14159 -1.5707 0" xyz="0 .04191 -.0306"/>
-      </visual>
-      <collision>
-        <geometry>
-          <mesh filename="package://robotiq_c_model_visualization/meshes/robotiq_85_gripper_joint_0_L.dae"/>
-        </geometry>
-        <origin rpy="3.14159 -1.5707 0" xyz="0 .04191 -.0306"/>
-      </collision>
-    </link>
-    <link name="robotiq_85_right_knuckle_link">
-      <inertial>
-        <mass value="10"/>
-        <origin xyz="0 0 0" rpy="0 0 0"/>
-        <inertia ixx="1" ixy="0" ixz="0" iyy="1" iyz="0" izz="1"/>
-      </inertial>
-      <visual>
-        <geometry>
-          <mesh filename="package://robotiq_c_model_visualization/meshes/robotiq_85_gripper_joint_0_R.dae"/>
-        </geometry>
-        <origin rpy="3.14159 1.5707 0" xyz="0 .04191 -.0306"/>
-      </visual>
-      <collision>
-        <geometry>
-          <mesh filename="package://robotiq_c_model_visualization/meshes/robotiq_85_gripper_joint_0_R.dae"/>
-        </geometry>
-        <origin rpy="3.14159 1.5707 0" xyz="0 .04191 -.0306"/>
-      </collision>
-    </link>
-    <!--  /\  -->
-    <!--  /\  -->
-    <joint name="robotiq_85_left_finger_joint" type="fixed">
-      <parent link="robotiq_85_left_knuckle_link"/>
-      <child link="robotiq_85_left_finger_link"/>
-      <axis xyz="1 0 0"/>
-      <origin rpy="3.1415 0 0" xyz="0 .00508 .03134"/>
-      <limit lower="0" upper="1.5707" velocity="2.0" effort="1000"/>
-    </joint>
-    <joint name="robotiq_85_right_finger_joint" type="fixed">
-      <parent link="robotiq_85_right_knuckle_link"/>
-      <child link="robotiq_85_right_finger_link"/>
-      <axis xyz="1 0 0"/>
-      <origin rpy="3.1415 0 0" xyz="0 .00508 .03134"/>
-      <limit lower="0" upper="1.5707" velocity="2.0" effort="1000"/>
-    </joint>
-    <!--  \/  -->
-    <!--  \/  -->
-    <link name="robotiq_85_left_finger_link">
-      <inertial>
-        <mass value="10"/>
-        <origin xyz="0 0 0" rpy="0 0 0"/>
-        <inertia ixx="1" ixy="0" ixz="0" iyy="1" iyz="0" izz="1"/>
-      </inertial>
-      <visual>
-        <geometry>
-          <mesh filename="package://robotiq_c_model_visualization/meshes/robotiq_85_gripper_joint_1_L.dae"/>
-        </geometry>
-        <origin rpy="0 1.5707 0" xyz="0 -.03683 .06194"/>
-      </visual>
-      <collision>
-        <geometry>
-          <mesh filename="package://robotiq_c_model_visualization/meshes/robotiq_85_gripper_joint_1_L.dae"/>
-        </geometry>
-        <origin rpy="0 1.5707 0" xyz="0 -.03683 .06194"/>
-      </collision>
-    </link>
-    <link name="robotiq_85_right_finger_link">
-      <inertial>
-        <mass value="10"/>
-        <origin xyz="0 0 0" rpy="0 0 0"/>
-        <inertia ixx="1" ixy="0" ixz="0" iyy="1" iyz="0" izz="1"/>
-      </inertial>
-      <visual>
-        <geometry>
-          <mesh filename="package://robotiq_c_model_visualization/meshes/robotiq_85_gripper_joint_1_R.dae"/>
-        </geometry>
-        <origin rpy="0 -1.5707 0" xyz="0 -.03683 .06194"/>
-      </visual>
-      <collision>
-        <geometry>
-          <mesh filename="package://robotiq_c_model_visualization/meshes/robotiq_85_gripper_joint_1_R.dae"/>
-        </geometry>
-        <origin rpy="0 -1.5707 0" xyz="0 -.03683 .06194"/>
-      </collision>
-    </link>
+    <xacro:if value="${hide_underactuated}">
+      <!--  /\  -->
+      <!--  /\  -->
+      <joint name="robotiq_85_left_knuckle_joint" type="revolute">
+        <parent link="robotiq_85_base_link"/>
+        <child link="robotiq_85_left_knuckle_link"/>
+        <axis xyz="1 0 0"/>
+        <origin rpy="-1.5707 1.5707 0" xyz=".04191 .0306 0"/>
+        <limit lower="0" upper=".8575" velocity="2.0" effort="1000"/>
+      </joint>
+      <joint name="robotiq_85_right_knuckle_joint" type="revolute">
+        <parent link="robotiq_85_base_link"/>
+        <child link="robotiq_85_right_knuckle_link"/>
+        <axis xyz="1 0 0"/>
+        <origin rpy="1.5707 -1.5707 0" xyz=".04191 -.0306 0"/>
+        <limit lower="0" upper="1.5707" velocity="2.0" effort="1000"/>
+        <xacro:if value="${hide_underactuated}">
+          <mimic joint="robotiq_85_left_knuckle_joint" multiplier="1"/>
+        </xacro:if>
+      </joint>
+      <!--  \/  -->
+      <!--  \/  -->
+      <link name="robotiq_85_left_knuckle_link">
+        <inertial>
+          <mass value="10"/>
+          <origin xyz="0 0 0" rpy="0 0 0"/>
+          <inertia ixx="1" ixy="0" ixz="0" iyy="1" iyz="0" izz="1"/>
+        </inertial>
+        <visual>
+          <geometry>
+            <mesh filename="package://robotiq_c_model_visualization/meshes/robotiq_85_gripper_joint_0_L.dae"/>
+          </geometry>
+          <origin rpy="3.14159 -1.5707 0" xyz="0 .04191 -.0306"/>
+        </visual>
+        <collision>
+          <geometry>
+            <mesh filename="package://robotiq_c_model_visualization/meshes/robotiq_85_gripper_joint_0_L.dae"/>
+          </geometry>
+          <origin rpy="3.14159 -1.5707 0" xyz="0 .04191 -.0306"/>
+        </collision>
+      </link>
+      <link name="robotiq_85_right_knuckle_link">
+        <inertial>
+          <mass value="10"/>
+          <origin xyz="0 0 0" rpy="0 0 0"/>
+          <inertia ixx="1" ixy="0" ixz="0" iyy="1" iyz="0" izz="1"/>
+        </inertial>
+        <visual>
+          <geometry>
+            <mesh filename="package://robotiq_c_model_visualization/meshes/robotiq_85_gripper_joint_0_R.dae"/>
+          </geometry>
+          <origin rpy="3.14159 1.5707 0" xyz="0 .04191 -.0306"/>
+        </visual>
+        <collision>
+          <geometry>
+            <mesh filename="package://robotiq_c_model_visualization/meshes/robotiq_85_gripper_joint_0_R.dae"/>
+          </geometry>
+          <origin rpy="3.14159 1.5707 0" xyz="0 .04191 -.0306"/>
+        </collision>
+      </link>
+      <!--  /\  -->
+      <!--  /\  -->
+      <joint name="robotiq_85_left_finger_joint" type="fixed">
+        <parent link="robotiq_85_left_knuckle_link"/>
+        <child link="robotiq_85_left_finger_link"/>
+        <axis xyz="1 0 0"/>
+        <origin rpy="3.1415 0 0" xyz="0 .00508 .03134"/>
+        <limit lower="0" upper="1.5707" velocity="2.0" effort="1000"/>
+      </joint>
+      <joint name="robotiq_85_right_finger_joint" type="fixed">
+        <parent link="robotiq_85_right_knuckle_link"/>
+        <child link="robotiq_85_right_finger_link"/>
+        <axis xyz="1 0 0"/>
+        <origin rpy="3.1415 0 0" xyz="0 .00508 .03134"/>
+        <limit lower="0" upper="1.5707" velocity="2.0" effort="1000"/>
+      </joint>
+      <!--  \/  -->
+      <!--  \/  -->
+      <link name="robotiq_85_left_finger_link">
+        <inertial>
+          <mass value="10"/>
+          <origin xyz="0 0 0" rpy="0 0 0"/>
+          <inertia ixx="1" ixy="0" ixz="0" iyy="1" iyz="0" izz="1"/>
+        </inertial>
+        <visual>
+          <geometry>
+            <mesh filename="package://robotiq_c_model_visualization/meshes/robotiq_85_gripper_joint_1_L.dae"/>
+          </geometry>
+          <origin rpy="0 1.5707 0" xyz="0 -.03683 .06194"/>
+        </visual>
+        <collision>
+          <geometry>
+            <mesh filename="package://robotiq_c_model_visualization/meshes/robotiq_85_gripper_joint_1_L.dae"/>
+          </geometry>
+          <origin rpy="0 1.5707 0" xyz="0 -.03683 .06194"/>
+        </collision>
+      </link>
+      <link name="robotiq_85_right_finger_link">
+        <inertial>
+          <mass value="10"/>
+          <origin xyz="0 0 0" rpy="0 0 0"/>
+          <inertia ixx="1" ixy="0" ixz="0" iyy="1" iyz="0" izz="1"/>
+        </inertial>
+        <visual>
+          <geometry>
+            <mesh filename="package://robotiq_c_model_visualization/meshes/robotiq_85_gripper_joint_1_R.dae"/>
+          </geometry>
+          <origin rpy="0 -1.5707 0" xyz="0 -.03683 .06194"/>
+        </visual>
+        <collision>
+          <geometry>
+            <mesh filename="package://robotiq_c_model_visualization/meshes/robotiq_85_gripper_joint_1_R.dae"/>
+          </geometry>
+          <origin rpy="0 -1.5707 0" xyz="0 -.03683 .06194"/>
+        </collision>
+      </link>
+    </xacro:if>
     <!--  /\  -->
     <!--  /\  -->
@@ -176,5 +180,7 @@
       <origin rpy="1.5707 1.5707 0" xyz=".04843 .0127 0"/>
       <limit lower="0" upper="1.5707" velocity="2.0" effort="1000"/>
-      <mimic joint="robotiq_85_left_knuckle_joint" offset="0"/>
+      <xacro:if value="${hide_underactuated}">
+        <mimic joint="robotiq_85_left_knuckle_joint" offset="0"/>
+      </xacro:if>
     </joint>
     <joint name="robotiq_85_right_inner_knuckle_joint" type="revolute">
@@ -184,5 +190,7 @@
       <origin rpy="-1.5707 -1.5707 0" xyz=".04843 -.0127 0"/>
       <limit lower="0" upper="1.5707" velocity="2.0" effort="1000"/>
-      <mimic joint="robotiq_85_left_knuckle_joint" offset="0"/>
+      <xacro:if value="${hide_underactuated}">
+        <mimic joint="robotiq_85_left_knuckle_joint" offset="0"/>
+      </xacro:if>
     </joint>
     <!--  \/  -->
@@ -234,5 +242,7 @@
       <origin rpy="0 0 0" xyz="0 .04196 -.0388"/>
       <limit lower="0" upper="1.5707" velocity="2.0" effort="1000"/>
-      <mimic joint="robotiq_85_left_knuckle_joint" multiplier="-1"/>
+      <xacro:if value="${hide_underactuated}">
+        <mimic joint="robotiq_85_left_knuckle_joint" multiplier="-1"/>
+      </xacro:if>
     </joint>
     <joint name="robotiq_85_right_finger_tip_joint" type="revolute">
@@ -242,5 +252,7 @@
       <origin rpy="0 0 0" xyz="0 .04196 -.0388"/>
       <limit lower="0" upper="1.5707" velocity="2.0" effort="1000"/>
-      <mimic joint="robotiq_85_left_knuckle_joint" multiplier="-1"/>
+      <xacro:if value="${hide_underactuated}">
+        <mimic joint="robotiq_85_left_knuckle_joint" multiplier="-1"/>
+      </xacro:if>
     </joint>
     <!--  \/  -->
@@ -284,116 +296,106 @@
       </collision>
     </link>
-    <transmission name="shoulder_pan_trans">
+    <xacro:if value="${hide_underactuated}">
+      <transmission name="robotiq_85_left_knuckle_trans">
+        <type>transmission_interface/SimpleTransmission</type>
+        <joint name="robotiq_85_left_knuckle_joint"/>
+        <actuator name="robotiq_85_left_knuckle_motor">
+          <hardwareInterface>PositionJointInterface</hardwareInterface>
+          <mechanicalReduction>1</mechanicalReduction>
+        </actuator>
+      </transmission>
+      <transmission name="robotiq_85_right_knuckle_trans">
+        <type>transmission_interface/SimpleTransmission</type>
+        <joint name="robotiq_85_right_knuckle_joint"/>
+        <actuator name="robotiq_85_right_knuckle_motor">
+          <hardwareInterface>PositionJointInterface</hardwareInterface>
+          <mechanicalReduction>1</mechanicalReduction>
+        </actuator>
+      </transmission>
+    </xacro:if>
+    <transmission name="robotiq_85_left_inner_knuckle_trans">
       <type>transmission_interface/SimpleTransmission</type>
-      <joint name="shoulder_pan_joint"/>
-      <actuator name="shoulder_pan_motor">
+      <joint name="robotiq_85_left_inner_knuckle_joint"/>
+      <actuator name="robotiq_85_left_inner_knuckle_motor">
         <hardwareInterface>PositionJointInterface</hardwareInterface>
         <mechanicalReduction>1</mechanicalReduction>
       </actuator>
     </transmission>
-    <transmission name="shoulder_lift_trans">
+    <transmission name="robotiq_85_right_inner_knuckle_trans">
       <type>transmission_interface/SimpleTransmission</type>
-      <joint name="shoulder_lift_joint"/>
-      <actuator name="shoulder_lift_motor">
+      <joint name="robotiq_85_right_inner_knuckle_joint"/>
+      <actuator name="robotiq_85_right_inner_knuckle_motor">
         <hardwareInterface>PositionJointInterface</hardwareInterface>
         <mechanicalReduction>1</mechanicalReduction>
       </actuator>
     </transmission>
-    <transmission name="elbow_trans">
+    <transmission name="robotiq_85_left_finger_tip_trans">
       <type>transmission_interface/SimpleTransmission</type>
-      <joint name="elbow_joint"/>
-      <actuator name="elbow_motor">
+      <joint name="robotiq_85_left_finger_tip_joint"/>
+      <actuator name="robotiq_85_left_finger_tip_motor">
         <hardwareInterface>PositionJointInterface</hardwareInterface>
         <mechanicalReduction>1</mechanicalReduction>
       </actuator>
     </transmission>
-    <transmission name="wrist_1_trans">
+    <transmission name="robotiq_85_right_finger_tip_trans">
       <type>transmission_interface/SimpleTransmission</type>
-      <joint name="wrist_1_joint"/>
-      <actuator name="wrist_1_motor">
+      <joint name="robotiq_85_right_finger_tip_joint"/>
+      <actuator name="robotiq_85_right_finger_tip_motor">
         <hardwareInterface>PositionJointInterface</hardwareInterface>
         <mechanicalReduction>1</mechanicalReduction>
       </actuator>
     </transmission>
-    <transmission name="wrist_2_trans">
-      <type>transmission_interface/SimpleTransmission</type>
-      <joint name="wrist_2_joint"/>
-      <actuator name="wrist_2_motor">
-        <hardwareInterface>PositionJointInterface</hardwareInterface>
-        <mechanicalReduction>1</mechanicalReduction>
-      </actuator>
-    </transmission>
-    <transmission name="wrist_3_trans">
-      <type>transmission_interface/SimpleTransmission</type>
-      <joint name="wrist_3_joint"/>
-      <actuator name="wrist_3_motor">
-        <hardwareInterface>PositionJointInterface</hardwareInterface>
-        <mechanicalReduction>1</mechanicalReduction>
-      </actuator>
-    </transmission>
-    <!-- <transmission name="robotiq_85_left_knuckle_trans">
-    <type>transmission_interface/SimpleTransmission</type>
-    <joint name="robotiq_85_left_knuckle_joint"/>
-    <actuator name="robotiq_85_left_knuckle_motor">
-      <hardwareInterface>PositionJointInterface</hardwareInterface>
-      <mechanicalReduction>1</mechanicalReduction>
-    </actuator>
-  </transmission>
-  <transmission name="robotiq_85_right_knuckle_trans">
-    <type>transmission_interface/SimpleTransmission</type>
-    <joint name="robotiq_85_right_knuckle_joint"/>
-    <actuator name="robotiq_85_right_knuckle_motor">
-      <hardwareInterface>PositionJointInterface</hardwareInterface>
-      <mechanicalReduction>1</mechanicalReduction>
-    </actuator>
-  </transmission>
-  <transmission name="robotiq_85_left_finger_trans">
-    <type>transmission_interface/SimpleTransmission</type>
-    <joint name="robotiq_85_left_finger_joint"/>
-    <actuator name="robotiq_85_left_finger_motor">
-      <hardwareInterface>PositionJointInterface</hardwareInterface>
-      <mechanicalReduction>1</mechanicalReduction>
-    </actuator>
-  </transmission>
-  <transmission name="robotiq_85_right_finger_trans">
-    <type>transmission_interface/SimpleTransmission</type>
-    <joint name="robotiq_85_right_finger_joint"/>
-    <actuator name="robotiq_85_right_finger_motor">
-      <hardwareInterface>PositionJointInterface</hardwareInterface>
-      <mechanicalReduction>1</mechanicalReduction>
-    </actuator>
-  </transmission>
-  <transmission name="robotiq_85_left_inner_knuckle_trans">
-    <type>transmission_interface/SimpleTransmission</type>
-    <joint name="robotiq_85_left_inner_knuckle_joint"/>
-    <actuator name="robotiq_85_left_inner_knuckle_motor">
-      <hardwareInterface>PositionJointInterface</hardwareInterface>
-      <mechanicalReduction>1</mechanicalReduction>
-    </actuator>
-  </transmission>
-  <transmission name="robotiq_85_right_inner_knuckle_trans">
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