Commit message: Added option to .xacro file, "hide_underactuated", to hide the outside "fingers" of the Robotiq gripper. Added back in the transmissions for the fingers to the robotiq URDF file, so that they show up correctly in RVIZ and so that MoveIt can plan. MoveIt cannot find valid positions for the gripper, so currently the gripper is disabled in ur5_robotiq_joint_limited.urdf.xacro.

File: ur5_robotiq_description/src/urdf/ur5_robotiq_joint_limited.urdf.xacro (robot description, xacro)
@@ -5,5 +5,7 @@
   <xacro:robot></xacro:robot>
   <xacro:include filename="$(find ur5_robotiq_description)/src/urdf/robotiq.urdf.xacro" />
-  <xacro:robotiq_c_model root_link="ee_fixed_link" ></xacro:robotiq_c_model>
+  <!--
+  <xacro:robotiq_c_model root_link="ee_fixed_link" hide_underactuated="false"></xacro:robotiq_c_model>
+  -->
   <!--
   <link name="world" />

Commit message: removing all references to fixed link

File: ur5_robotiq_description/src/urdf/base_ur5.urdf.xacro (robot description, xacro)
@@ -212,8 +212,8 @@
   <joint name="ee_fixed_joint" type="fixed">
     <parent link="wrist_3_link"/>
-    <child link="ee_fixed_link"/>
+    <child link="ee_link"/>
     <origin rpy="0.0 0.0 1.570796325" xyz="0.0 0.0823 0.0"/>
   </joint>
-  <link name="ee_fixed_link"/>
+  <link name="ee_link"/>
   <transmission name="shoulder_pan_trans">
     <type>transmission_interface/SimpleTransmission</type>

File: ur5_robotiq_description/src/urdf/ur5_robotiq_joint_limited.urdf (robot description, URDF)
Before this commit: robot ur5, 9 links, 8 joints
Links:
- removed link ee_fixed_link
- added link ee_link
Joints:
- joint ee_fixed_joint: child ee_fixed_link -> ee_link

File: ur5_robotiq_description/src/urdf/ur5_robotiq_joint_limited.urdf.xacro (robot description, xacro)
@@ -5,10 +5,10 @@
   <xacro:robot></xacro:robot>
   <!-- <xacro:include filename="$(find ur5_robotiq_description)/src/urdf/robotiq.urdf.xacro" /> -->
-  <xacro:robotiq_c_model root_link="ee_fixed_link" show_underactuated="false" gravity="false"></xacro:robotiq_c_model>
+  <xacro:robotiq_c_model root_link="ee_link" show_underactuated="false" gravity="false"></xacro:robotiq_c_model>
   <!--
   <xacro:include filename="$(find ur5_robotiq_description)/src/urdf/s_model/s-model_articulated_macro.xacro"/>
   <xacro:s-model_articulated prefix=""></xacro:s-model_articulated>
   <joint name="s_model_to_arm" type="fixed">
-    <parent link="ee_fixed_link"/>
+    <parent link="ee_link"/>
     <child link="palm"/>
     <origin rpy="0.0 0.0 0.0" xyz="0.0 0.1363 0.0"/>

File: ur_description/urdf/ur5_joint_limited.urdf.xacro (robot description, xacro)
@@ -222,8 +222,8 @@
   <joint name="${prefix}ee_fixed_joint" type="fixed">
     <parent link="${prefix}wrist_3_link" />
-    <child link = "${prefix}ee_fixed_link" />
+    <child link = "${prefix}ee_link" />
     <origin xyz="0.0 ${wrist_3_length} 0.0" rpy="0.0 0.0 ${pi/2.0}" />
   </joint>
-  <link name="${prefix}ee_fixed_link" />
+  <link name="${prefix}ee_link" />
   <link name="${prefix}gripper_link">
     <visual>
@@ -281,5 +281,5 @@
   </link>
   <joint name="${prefix}ee_link_gripper" type="fixed">
-    <parent link="${prefix}ee_fixed_link"/>
+    <parent link="${prefix}ee_link"/>
     <child link="${prefix}gripper_link"/>
     <origin rpy="${pi/2} ${pi/2} ${pi/2}" xyz="0.05 0 0"/>

File: ur_description/urdf/ur5_robot.urdf (robot description, URDF)
Before this commit: robot ur5, 8 links, 7 joints
Links:
- removed link ee_fixed_link
- added link ee_link
Joints:
- joint ee_fixed_joint: child ee_fixed_link -> ee_link
