Commit message: fixed cartesian endpoint control with the marker_teleop interface

File: ur_description/urdf/ur5.urdf.xacro (robot description, xacro)
@@ -49,5 +49,6 @@
 		    <mesh filename="package://ur_description/meshes/ur5/visual/Base.dae" />
       </geometry>
-      <origin xyz="0.0 0.0 0.003" rpy="0.0 0.0 ${3.0 * pi / 4.0}" />
+      <!-- <origin xyz="0.0 0.0 0.003" rpy="0.0 0.0 ${3.0 * pi / 4.0}" /> -->
+      <origin xyz="0.0 0.0 0.003" rpy="0.0 0.0 ${-pi/4.0}" />
     </visual>
 	<collision>
@@ -65,5 +66,6 @@
     <parent link="${prefix}base_link" />
     <child link = "${prefix}shoulder_link" />
-    <origin xyz="0.0 0.0 ${shoulder_height}" rpy="0.0 0.0 0.0" />
+    <!-- <origin xyz="0.0 0.0 ${shoulder_height}" rpy="0.0 0.0 0.0" /> -->
+    <origin xyz="0.0 0.0 ${shoulder_height}" rpy="0.0 0.0 3.1415" />
     <axis xyz="0 0 1" />
     <limit lower="${-2.0 * pi}" upper="${2.0 * pi}" effort="150.0" velocity="${pi}"/>

Commit message: removed comments from xacro file

File: ur_description/urdf/ur5.urdf.xacro (robot description, xacro)
@@ -49,5 +49,4 @@
 		    <mesh filename="package://ur_description/meshes/ur5/visual/Base.dae" />
       </geometry>
-      <!-- <origin xyz="0.0 0.0 0.003" rpy="0.0 0.0 ${3.0 * pi / 4.0}" /> -->
       <origin xyz="0.0 0.0 0.003" rpy="0.0 0.0 ${-pi/4.0}" />
     </visual>
@@ -66,5 +65,4 @@
     <parent link="${prefix}base_link" />
     <child link = "${prefix}shoulder_link" />
-    <!-- <origin xyz="0.0 0.0 ${shoulder_height}" rpy="0.0 0.0 0.0" /> -->
     <origin xyz="0.0 0.0 ${shoulder_height}" rpy="0.0 0.0 3.1415" />
     <axis xyz="0 0 1" />

Commit message: our changes to these files

File: ur_description/urdf/ur5.urdf.xacro (robot description, xacro)
@@ -146,5 +146,5 @@
     <origin xyz="0.0 0.0 ${forearm_length}" rpy="0.0 ${pi / 2.0} 0.0" />
     <axis xyz="0 1 0" />
-    <limit lower="${-1.0 * pi}" upper="${0.25 * pi}" effort="28.0" velocity="${pi}"/>
+    <limit lower="${-2.0 * pi}" upper="${2.0 * pi}" effort="28.0" velocity="${pi}"/>
     <dynamics damping="0.3" friction="0.0"/>
   </joint>
@@ -226,5 +226,6 @@
   </joint>
   <link name="${prefix}ee_link" />
-  <xacro:ur5_arm_transmission prefix="${prefix}" />
+  <!-- Change to fix urdf_parse_error -->
+  <!-- <xacro:ur5_arm_transmission prefix="${prefix}" /> -->
   <xacro:ur5_arm_gazebo prefix="${prefix}" />
   </xacro:macro>

File: ur_description/urdf/ur5_joint_limited.urdf.xacro (robot description, xacro)
@@ -226,5 +226,6 @@
   </joint>
   <link name="${prefix}ee_fixed_link" />
-  <xacro:ur5_arm_transmission prefix="${prefix}" />
+  <!-- Change to fix urdf_parse_error -->
+  <!-- <xacro:ur5_arm_transmission prefix="${prefix}" /> -->
   <xacro:ur5_arm_gazebo prefix="${prefix}" />
   </xacro:macro>
