Commit message: joint limited ur5 is now correct: lines up with driver, other urdf

File: ur_description/urdf/ur5_joint_limited.urdf.xacro (robot description, xacro)
@@ -49,5 +49,5 @@
 		    <mesh filename="package://ur_description/meshes/ur5/visual/Base.dae" />
       </geometry>
-      <origin xyz="0.0 0.0 0.003" rpy="0.0 0.0 ${3.0 * pi / 4.0}" />
+      <origin xyz="0.0 0.0 0.003" rpy="0.0 0.0 ${-1.0 * pi / 4.0}" />
     </visual>
 	<collision>
@@ -65,5 +65,5 @@
     <parent link="${prefix}base_link" />
     <child link = "${prefix}shoulder_link" />
-    <origin xyz="0.0 0.0 ${shoulder_height}" rpy="0.0 0.0 0.0" />
+    <origin xyz="0.0 0.0 ${shoulder_height}" rpy="0.0 0.0 3.1415" />
     <axis xyz="0 0 1" />
     <limit lower="${-pi}" upper="${pi}" effort="150.0" velocity="${pi}"/>

Commit message: changed joint limits

File: ur_description/urdf/ur5_joint_limited.urdf.xacro (robot description, xacro)
@@ -146,5 +146,5 @@
     <origin xyz="0.0 0.0 ${forearm_length}" rpy="0.0 ${pi / 2.0} 0.0" />
     <axis xyz="0 1 0" />
-    <limit lower="${-1.0 * pi}" upper="${0.25 * pi}" effort="28.0" velocity="${pi}"/>
+    <limit lower="${-1.0 * pi}" upper="${pi}" effort="28.0" velocity="${pi}"/>
     <dynamics damping="0.3" friction="0.0"/>
   </joint>
@@ -226,4 +226,63 @@
   </joint>
   <link name="${prefix}ee_fixed_link" />
+  <link name="${prefix}gripper_link">
+    <visual>
+      <geometry>
+        <cylinder length="0.09" radius="0.065"/>
+      </geometry>
+      <origin rpy="0 0 0" xyz="0 0 0"/>
+      <material name="white"/>
+    </visual>
+    <visual>
+      <geometry>
+        <box size="0.15 0.02 0.04"/>
+      </geometry>
+      <origin rpy="0 0 0" xyz="0 0 0.065"/>
+      <material name="blue"/>
+    </visual>
+    <visual>
+      <geometry>
+        <box size="0.03 0.02 0.05"/>
+      </geometry>
+      <origin rpy="0 0 0" xyz="-0.06 0 0.11"/>
+      <material name="white"/>
+    </visual>
+    <visual>
+      <geometry>
+        <box size="0.03 0.02 0.05"/>
+      </geometry>
+      <origin rpy="0 0 0" xyz="0.06 0 0.11"/>
+      <material name="white"/>
+    </visual>
+    <collision>
+      <geometry>
+        <cylinder length="0.09" radius="0.065"/>
+      </geometry>
+      <origin rpy="0 0 0" xyz="0 0 0"/>
+    </collision>
+    <collision>
+      <geometry>
+        <box size="0.15 0.02 0.04"/>
+      </geometry>
+      <origin rpy="0 0 0" xyz="0 0 0.065"/>
+    </collision>
+    <collision>
+      <geometry>
+        <box size="0.03 0.02 0.05"/>
+      </geometry>
+      <origin rpy="0 0 0" xyz="-0.06 0 0.11"/>
+    </collision>
+    <collision>
+      <geometry>
+        <box size="0.03 0.02 0.05"/>
+      </geometry>
+      <origin rpy="0 0 0" xyz="0.06 0 0.11"/>
+    </collision>
+  </link>
+  <joint name="${prefix}ee_link_gripper" type="fixed">
+    <parent link="${prefix}ee_fixed_link"/>
+    <child link="${prefix}gripper_link"/>
+    <origin rpy="${pi/2} ${pi/2} ${pi/2}" xyz="0.05 0 0"/>
+  </joint>
   <!-- Change to fix urdf_parse_error -->
   <!-- <xacro:ur5_arm_transmission prefix="${prefix}" /> -->

Commit message: ...

File: ur_description/urdf/ur5_joint_limited.urdf.xacro (robot description, xacro)
@@ -232,5 +232,5 @@
       </geometry>
       <origin rpy="0 0 0" xyz="0 0 0"/>
-      <material name="white"/>
+      <material name="White"/>
     </visual>
     <visual>
@@ -239,5 +239,5 @@
       </geometry>
       <origin rpy="0 0 0" xyz="0 0 0.065"/>
-      <material name="blue"/>
+      <material name="LightGrey"/>
     </visual>
     <visual>
@@ -246,5 +246,5 @@
       </geometry>
       <origin rpy="0 0 0" xyz="-0.06 0 0.11"/>
-      <material name="white"/>
+      <material name="White"/>
     </visual>
     <visual>
@@ -253,5 +253,5 @@
       </geometry>
       <origin rpy="0 0 0" xyz="0.06 0 0.11"/>
-      <material name="white"/>
+      <material name="White"/>
     </visual>
     <collision>
