Commit message: corrected the relative pose between fixture_3 and wrist_2_link & added collision detection waiver for fixutre_1, fixture_2 and fixture_3

File: ur_description/urdf/ur5_fixture.urdf.xacro (robot description, xacro)
@@ -138,4 +138,7 @@
                   <cylinder radius="0.023" length="0.07"/>
               </geometry>
+              <material name="FixtureColor">
+                  <color rgba="0.2 0.2 1 1"/>
+              </material>
           </visual>
           <collision>
@@ -145,4 +148,7 @@
                   <cylinder radius="0.023" length="0.07"/>
               </geometry>
+              <material name="White">
+                  <color rgba="1 1 1 1"/>
+              </material>
           </collision>
       </link>
@@ -191,4 +197,7 @@
                   <cylinder radius="0.023" length="0.07"/>
               </geometry>
+              <material name="FixtureColor">
+                  <color rgba="0.2 0.2 1 1"/>
+              </material>
           </visual>
           <collision>
@@ -268,26 +277,4 @@
           <dynamics damping="0.0" friction="0.0"/>
       </joint>
-       <link name="${prefix}fixture_3_link">
-          <visual>
-              <origin xyz="-0.06278 -0.026 -0.03625" rpy="0 1.04719 0"/>
-              <geometry>
-                  <!-- CAD measured -->
-                  <cylinder radius="0.023" length="0.07"/>
-              </geometry>
-          </visual>
-          <collision>
-              <origin xyz="-0.06278 -0.026 -0.03625" rpy="0 1.04719 0"/>
-              <geometry>
-                  <!-- CAD measured -->
-                  <cylinder radius="0.023" length="0.07"/>
-              </geometry>
-          </collision>
-      </link>
-      <joint name="${prefix}wrist_1_fixture_joint" type="fixed">
-          <parent link="${prefix}wrist_1_link" />
-          <child link = "${prefix}fixture_3_link" />
-          <origin xyz="0.0 0.0 0.0" rpy="0.0 0.0 0.0" />
-          <axis xyz="0 0 1" />
-      </joint>
       <link name="${prefix}wrist_2_link">
           <visual>
@@ -343,4 +330,33 @@
           <child link = "${prefix}ee_link" />
           <origin xyz="0.0 ${wrist_3_length} 0.0" rpy="0.0 0.0 ${pi/2.0}" />
+      </joint>
+      <link name="${prefix}fixture_3_link">
+          <visual>
+              <!-- origin xyz="-0.03625  -0.026 0.06278" rpy="0 -0.52359 0"/-->
+              <origin xyz="-0.03625  -0.026 0.15578" rpy="0 -0.52359 0"/>
+              <geometry>
+                  <!-- CAD measured -->
+                  <cylinder radius="0.023" length="0.07"/>
+              </geometry>
+              <material name="FixtureColor">
+                  <color rgba="0.2 0.2 1 1"/>
+              </material>
+          </visual>
+          <collision>
+              <origin xyz="-0.03625  -0.026 0.15578" rpy="0 -0.52359 0"/>
+              <geometry>
+                  <!-- CAD measured -->
+                  <cylinder radius="0.023" length="0.07"/>
+              </geometry>
+              <material name="White">
+                  <color rgba="1 1 1 1"/>
+              </material>
+          </collision>
+      </link>
+      <joint name="${prefix}wrist_2_fixture_joint" type="fixed">
+          <parent link="${prefix}wrist_2_link" />
+          <child link = "${prefix}fixture_3_link" />
+          <origin xyz="0.0 0.0 0.0" rpy="0.0 0.0 0.0" />
+          <axis xyz="0 0 1" />
       </joint>
       <link name="${prefix}ee_link">
@@ -359,17 +375,16 @@
           <!-- NOTE: this rotation is only needed as long as base_link itself is
                  not corrected wrt the real robot (ie: rotated over 180
-                 degrees)
-      -->
-      <origin xyz="0 0 0" rpy="0 0 ${-pi}"/>
-      <parent link="${prefix}base_link"/>
-      <child link="${prefix}base"/>
-  </joint>
-  <!-- Frame coincident with all-zeros TCP on UR controller -->
-  <link name="${prefix}tool0"/>
-  <joint name="${prefix}wrist_3_link-tool0_fixed_joint" type="fixed">
-      <origin xyz="0 ${wrist_3_length} 0" rpy="${pi/-2.0} 0 0"/>
-      <parent link="${prefix}wrist_3_link"/>
-      <child link="${prefix}tool0"/>
-  </joint>
-  </xacro:macro>
+                 degrees)-->
+        <origin xyz="0 0 0" rpy="0 0 ${-pi}"/>
+        <parent link="${prefix}base_link"/>
+        <child link="${prefix}base"/>
+    </joint>
+    <!-- Frame coincident with all-zeros TCP on UR controller -->
+    <link name="${prefix}tool0"/>
+    <joint name="${prefix}wrist_3_link-tool0_fixed_joint" type="fixed">
+        <origin xyz="0 ${wrist_3_length} 0" rpy="${pi/-2.0} 0 0"/>
+        <parent link="${prefix}wrist_3_link"/>
+        <child link="${prefix}tool0"/>
+    </joint>
+</xacro:macro>
 </robot>

Commit message: changes to get the joint planner to work

File: ur_description/urdf/ur5_fixture.urdf.xacro (robot description, xacro)
@@ -96,5 +96,5 @@
           </xacro:unless>
           <xacro:if value="${joint_limited}">
-              <limit lower="${-pi}" upper="${pi}" effort="150.0" velocity="3.15"/>
+              <limit lower="${-2*pi}" upper="${2*pi}" effort="150.0" velocity="3.15"/>
           </xacro:if>
           <dynamics damping="0.0" friction="0.0"/>
@@ -127,5 +127,5 @@
           </xacro:unless>
           <xacro:if value="${joint_limited}">
-              <limit lower="${-pi}" upper="${pi}" effort="150.0" velocity="3.15"/>
+              <limit lower="${-2*pi}" upper="${2*pi}" effort="150.0" velocity="3.15"/>
           </xacro:if>
           <dynamics damping="0.0" friction="0.0"/>
@@ -186,5 +186,5 @@
           </xacro:unless>
           <xacro:if value="${joint_limited}">
-              <limit lower="${-pi}" upper="${pi}" effort="150.0" velocity="3.15"/>
+              <limit lower="${-2*pi}" upper="${2*pi}" effort="150.0" velocity="3.15"/>
           </xacro:if>
           <dynamics damping="0.0" friction="0.0"/>
@@ -242,5 +242,5 @@
           </xacro:unless>
           <xacro:if value="${joint_limited}">
-              <limit lower="${-pi}" upper="${pi}" effort="28.0" velocity="3.2"/>
+              <limit lower="${-2*pi}" upper="${2*pi}" effort="28.0" velocity="3.2"/>
           </xacro:if>
           <dynamics damping="0.0" friction="0.0"/>
@@ -273,5 +273,5 @@
           </xacro:unless>
           <xacro:if value="${joint_limited}">
-              <limit lower="${-pi}" upper="${pi}" effort="28.0" velocity="3.2"/>
+              <limit lower="${-2*pi}" upper="${2*pi}" effort="28.0" velocity="3.2"/>
           </xacro:if>
           <dynamics damping="0.0" friction="0.0"/>
@@ -304,5 +304,5 @@
           </xacro:unless>
           <xacro:if value="${joint_limited}">
-              <limit lower="${-pi}" upper="${pi}" effort="28.0" velocity="3.2"/>
+              <limit lower="${-2*pi}" upper="${2*pi}" effort="28.0" velocity="3.2"/>
           </xacro:if>
           <dynamics damping="0.0" friction="0.0"/>

Commit message: changed back limited joint ranges to their original settings

File: ur_description/urdf/ur5_fixture.urdf.xacro (robot description, xacro)
@@ -96,5 +96,5 @@
           </xacro:unless>
           <xacro:if value="${joint_limited}">
-              <limit lower="${-2*pi}" upper="${2*pi}" effort="150.0" velocity="3.15"/>
+              <limit lower="${-pi}" upper="${pi}" effort="150.0" velocity="3.15"/>
           </xacro:if>
           <dynamics damping="0.0" friction="0.0"/>
@@ -127,5 +127,5 @@
           </xacro:unless>
           <xacro:if value="${joint_limited}">
-              <limit lower="${-2*pi}" upper="${2*pi}" effort="150.0" velocity="3.15"/>
+              <limit lower="${-pi}" upper="${pi}" effort="150.0" velocity="3.15"/>
           </xacro:if>
           <dynamics damping="0.0" friction="0.0"/>
@@ -186,5 +186,5 @@
           </xacro:unless>
           <xacro:if value="${joint_limited}">
-              <limit lower="${-2*pi}" upper="${2*pi}" effort="150.0" velocity="3.15"/>
+              <limit lower="${-pi}" upper="${pi}" effort="150.0" velocity="3.15"/>
           </xacro:if>
           <dynamics damping="0.0" friction="0.0"/>
@@ -242,5 +242,5 @@
           </xacro:unless>
           <xacro:if value="${joint_limited}">
-              <limit lower="${-2*pi}" upper="${2*pi}" effort="28.0" velocity="3.2"/>
+              <limit lower="${-pi}" upper="${pi}" effort="28.0" velocity="3.2"/>
           </xacro:if>
           <dynamics damping="0.0" friction="0.0"/>
@@ -273,5 +273,5 @@
           </xacro:unless>
           <xacro:if value="${joint_limited}">
-              <limit lower="${-2*pi}" upper="${2*pi}" effort="28.0" velocity="3.2"/>
+              <limit lower="${-pi}" upper="${pi}" effort="28.0" velocity="3.2"/>
           </xacro:if>
           <dynamics damping="0.0" friction="0.0"/>
@@ -304,5 +304,5 @@
           </xacro:unless>
           <xacro:if value="${joint_limited}">
-              <limit lower="${-2*pi}" upper="${2*pi}" effort="28.0" velocity="3.2"/>
+              <limit lower="${-pi}" upper="${pi}" effort="28.0" velocity="3.2"/>
           </xacro:if>
           <dynamics damping="0.0" friction="0.0"/>

Commit message: changed the joint limits for limited=false such that they are consistent with the soft limits in the driver

File: ur_description/urdf/ur5_fixture.urdf.xacro (robot description, xacro)
@@ -93,5 +93,7 @@
           <axis xyz="0 0 1" />
           <xacro:unless value="${joint_limited}">
-              <limit lower="${-2.0 * pi}" upper="${2.0 * pi}" effort="150.0" velocity="3.15"/>
+              <!-- limit lower="${-2.0 * pi}" upper="${2.0 * pi}" effort="150.0" velocity="3.15"/-->
+              <!-- Set as the soft joint limits as in the driver -->
+              <limit lower="${-6.05}" upper="${6.05}" effort="150.0" velocity="3.15"/>
           </xacro:unless>
           <xacro:if value="${joint_limited}">
@@ -124,5 +126,7 @@
           <axis xyz="0 1 0" />
           <xacro:unless value="${joint_limited}">
-              <limit lower="${-2.0 * pi}" upper="${2.0 * pi}" effort="150.0" velocity="3.15"/>
+              <!-- limit lower="${-2.0 * pi}" upper="${2.0 * pi}" effort="150.0" velocity="3.15"/-->
+              <!-- Set as the soft joint limits as in the driver -->
+              <limit lower="${-6.05}" upper="${6.05}" effort="150.0" velocity="3.15"/>
           </xacro:unless>
           <xacro:if value="${joint_limited}">
@@ -183,5 +187,7 @@
           <axis xyz="0 1 0" />
           <xacro:unless value="${joint_limited}">
-              <limit lower="${-2.0 * pi}" upper="${2.0 * pi}" effort="150.0" velocity="3.15"/>
+              <!-- limit lower="${-2.0 * pi}" upper="${2.0 * pi}" effort="150.0" velocity="3.15"/-->
+              <!-- Set as the soft joint limits as in the driver -->
+              <limit lower="${-6.05}" upper="${6.05}" effort="150.0" velocity="3.15"/>
           </xacro:unless>
           <xacro:if value="${joint_limited}">
@@ -239,5 +245,7 @@
           <axis xyz="0 1 0" />
           <xacro:unless value="${joint_limited}">
-              <limit lower="${-2.0 * pi}" upper="${2.0 * pi}" effort="28.0" velocity="3.2"/>
+              <!-- limit lower="${-2.0 * pi}" upper="${2.0 * pi}" effort="28.0" velocity="3.2"/-->
+              <!-- Set as the soft joint limits as in the driver -->
+              <limit lower="${-6.05}" upper="${6.05}" effort="150.0" velocity="3.15"/>
           </xacro:unless>
           <xacro:if value="${joint_limited}">
@@ -270,5 +278,7 @@
           <axis xyz="0 0 1" />
           <xacro:unless value="${joint_limited}">
-              <limit lower="${-2.0 * pi}" upper="${2.0 * pi}" effort="28.0" velocity="3.2"/>
+              <!-- limit lower="${-2.0 * pi}" upper="${2.0 * pi}" effort="28.0" velocity="3.2"/-->
+              <!-- Set as the soft joint limits as in the driver -->
+              <limit lower="${-6.05}" upper="${6.05}" effort="150.0" velocity="3.15"/>
           </xacro:unless>
           <xacro:if value="${joint_limited}">
@@ -301,5 +311,7 @@
           <axis xyz="0 1 0" />
           <xacro:unless value="${joint_limited}">
-              <limit lower="${-2.0 * pi}" upper="${2.0 * pi}" effort="28.0" velocity="3.2"/>
+              <!-- limit lower="${-2.0 * pi}" upper="${2.0 * pi}" effort="28.0" velocity="3.2"/-->
+              <!-- Set as the soft joint limits as in the driver -->
+              <limit lower="${-6.05}" upper="${6.05}" effort="150.0" velocity="3.15"/>
           </xacro:unless>
           <xacro:if value="${joint_limited}">
