Commit message: Fix/1262 (#9)
* changed world frame to stand

* removing / from tf lookups

File: ur_description/urdf/ur10_joint_limited_robot.urdf.xacro (robot description, xacro)
@@ -8,7 +8,7 @@
   <!-- arm -->
   <xacro:ur10_robot prefix="" joint_limited="true"/>
-  <link name="world" />
+  <link name="stand" />
   <joint name="world_joint" type="fixed">
-    <parent link="world" />
+    <parent link="stand" />
     <child link = "base_link" />
     <origin xyz="0.0 0.0 0.0" rpy="0.0 0.0 0.0" />

File: ur_description/urdf/ur10_robot.urdf.xacro (robot description, xacro)
@@ -8,7 +8,7 @@
   <!-- arm -->
   <xacro:ur10_robot prefix="" joint_limited="false"/>
-  <link name="world" />
+  <link name="stand" />
   <joint name="world_joint" type="fixed">
-    <parent link="world" />
+    <parent link="stand" />
     <child link = "base_link" />
     <origin xyz="0.0 0.0 0.0" rpy="0.0 0.0 0.0" />

File: ur_description/urdf/ur3_joint_limited_robot.urdf.xacro (robot description, xacro)
@@ -8,7 +8,7 @@
   <!-- arm -->
   <xacro:ur3_robot prefix="" joint_limited="true"/>
-  <link name="world" />
+  <link name="stand" />
   <joint name="world_joint" type="fixed">
-    <parent link="world" />
+    <parent link="stand" />
     <child link = "base_link" />
     <origin xyz="0.0 0.0 0.0" rpy="0.0 0.0 0.0" />

File: ur_description/urdf/ur3_robot.urdf.xacro (robot description, xacro)
@@ -8,7 +8,7 @@
   <!-- arm -->
   <xacro:ur3_robot prefix="" joint_limited="false"/>
-  <link name="world" />
+  <link name="stand" />
   <joint name="world_joint" type="fixed">
-    <parent link="world" />
+    <parent link="stand" />
     <child link = "base_link" />
     <origin xyz="0.0 0.0 0.0" rpy="0.0 0.0 0.0" />

File: ur_description/urdf/ur5_joint_limited_robot.urdf.xacro (robot description, xacro)
@@ -8,7 +8,7 @@
   <!-- arm -->
   <xacro:ur5_robot prefix="" joint_limited="true"/>
-  <link name="world" />
+  <link name="stand" />
   <joint name="world_joint" type="fixed">
-    <parent link="world" />
+    <parent link="stand" />
     <child link = "base_link" />
     <origin xyz="0.0 0.0 0.0" rpy="0.0 0.0 0.0" />

File: ur_description/urdf/ur5_robot.urdf.xacro (robot description, xacro)
@@ -8,7 +8,7 @@
   <!-- arm -->
   <xacro:ur5_robot prefix="" joint_limited="false"/>
-  <link name="world" />
+  <link name="stand" />
   <joint name="world_joint" type="fixed">
-    <parent link="world" />
+    <parent link="stand" />
     <child link = "base_link" />
     <origin xyz="0.0 0.0 0.0" rpy="0.0 0.0 0.0" />
