Commit message: Stash this away for now

File: ur_description/urdf/ur5e.urdf.xacro (robot description, xacro)
@@ -43,10 +43,10 @@
   joint_direction = [1, 1, -1, 1, 1, 1]
   -->
-  <property name="ur5_a2" value="-0.42500" />
-  <property name="ur5_a3" value="-0.39220" />
-  <property name="ur5_d1" value="0.1625" />
-  <property name="ur5_d4" value="0.1333" />
-  <property name="ur5_d5" value="0.09970" />
-  <property name="ur5_d6" value="0.0996" />
+  <property name="ur5e_a2" value="-0.42500" />
+  <property name="ur5e_a3" value="-0.39220" />
+  <property name="ur5e_d1" value="0.1625" />
+  <property name="ur5e_d4" value="0.1333" />
+  <property name="ur5e_d5" value="0.09970" />
+  <property name="ur5e_d6" value="0.0996" />
   <!-- Properties from urcontrol.conf.UR5 e-series -->
   <!--
@@ -68,10 +68,10 @@
   <property name="elbow_offset" value="0.093" />
   <!-- Link lengths used in model -->
-  <property name="shoulder_height" value="${ur5_d1}" />
-  <property name="upper_arm_length" value="${-ur5_a2}" />
-  <property name="forearm_length" value="${-ur5_a3}" />
-  <property name="wrist_1_length" value="${ur5_d4 - elbow_offset - shoulder_offset}" />
-  <property name="wrist_2_length" value="${ur5_d5}" />
-  <property name="wrist_3_length" value="${ur5_d6}" />
+  <property name="shoulder_height" value="${ur5e_d1}" />
+  <property name="upper_arm_length" value="${-ur5e_a2}" />
+  <property name="forearm_length" value="${-ur5e_a3}" />
+  <property name="wrist_1_length" value="${ur5e_d4 - elbow_offset - shoulder_offset}" />
+  <property name="wrist_2_length" value="${ur5e_d5}" />
+  <property name="wrist_3_length" value="${ur5e_d6}" />
   <xacro:macro name="cylinder_inertial" params="radius length mass *origin">
     <inertial>
@@ -83,17 +83,17 @@
     </inertial>
   </xacro:macro>
-  <xacro:macro name="ur5_robot" params="prefix joint_limited">
+  <xacro:macro name="ur5e_robot" params="prefix joint_limited">
     <link name="${prefix}base_link" >
       <visual>
         <geometry>
-          <mesh filename="package://ur_description/meshes/ur5/visual/base.dae" />
-        </geometry>
-        <material name="LightGrey">
-          <color rgba="0.7 0.7 0.7 1.0"/>
-        </material>
-      </visual>
-      <collision>
-        <geometry>
-          <mesh filename="package://ur_description/meshes/ur5/collision/base.stl" />
+          <mesh filename="package://ur_description/meshes/ur5e/visual/base.dae" />
+        </geometry>
+        <material name="LightGrey">
+          <color rgba="0.7 0.7 0.7 1.0"/>
+        </material>
+      </visual>
+      <collision>
+        <geometry>
+          <mesh filename="package://ur_description/meshes/ur5e/collision/base.stl" />
         </geometry>
       </collision>
@@ -118,13 +118,13 @@
       <visual>
         <geometry>
-          <mesh filename="package://ur_description/meshes/ur5/visual/shoulder.dae" />
-        </geometry>
-        <material name="LightGrey">
-          <color rgba="0.7 0.7 0.7 1.0"/>
-        </material>
-      </visual>
-      <collision>
-        <geometry>
-          <mesh filename="package://ur_description/meshes/ur5/collision/shoulder.stl" />
+          <mesh filename="package://ur_description/meshes/ur5e/visual/shoulder.dae" />
+        </geometry>
+        <material name="LightGrey">
+          <color rgba="0.7 0.7 0.7 1.0"/>
+        </material>
+      </visual>
+      <collision>
+        <geometry>
+          <mesh filename="package://ur_description/meshes/ur5e/collision/shoulder.stl" />
         </geometry>
       </collision>
@@ -149,13 +149,13 @@
       <visual>
         <geometry>
-          <mesh filename="package://ur_description/meshes/ur5/visual/upperarm.dae" />
-        </geometry>
-        <material name="LightGrey">
-          <color rgba="0.7 0.7 0.7 1.0"/>
-        </material>
-      </visual>
-      <collision>
-        <geometry>
-          <mesh filename="package://ur_description/meshes/ur5/collision/upperarm.stl" />
+          <mesh filename="package://ur_description/meshes/ur5e/visual/upperarm.dae" />
+        </geometry>
+        <material name="LightGrey">
+          <color rgba="0.7 0.7 0.7 1.0"/>
+        </material>
+      </visual>
+      <collision>
+        <geometry>
+          <mesh filename="package://ur_description/meshes/ur5e/collision/upperarm.stl" />
         </geometry>
       </collision>
@@ -180,13 +180,13 @@
       <visual>
         <geometry>
-          <mesh filename="package://ur_description/meshes/ur5/visual/forearm.dae" />
-        </geometry>
-        <material name="LightGrey">
-          <color rgba="0.7 0.7 0.7 1.0"/>
-        </material>
-      </visual>
-      <collision>
-        <geometry>
-          <mesh filename="package://ur_description/meshes/ur5/collision/forearm.stl" />
+          <mesh filename="package://ur_description/meshes/ur5e/visual/forearm.dae" />
+        </geometry>
+        <material name="LightGrey">
+          <color rgba="0.7 0.7 0.7 1.0"/>
+        </material>
+      </visual>
+      <collision>
+        <geometry>
+          <mesh filename="package://ur_description/meshes/ur5e/collision/forearm.stl" />
         </geometry>
       </collision>
@@ -211,13 +211,13 @@
       <visual>
         <geometry>
-          <mesh filename="package://ur_description/meshes/ur5/visual/wrist1.dae" />
-        </geometry>
-        <material name="LightGrey">
-          <color rgba="0.7 0.7 0.7 1.0"/>
-        </material>
-      </visual>
-      <collision>
-        <geometry>
-          <mesh filename="package://ur_description/meshes/ur5/collision/wrist1.stl" />
+          <mesh filename="package://ur_description/meshes/ur5e/visual/wrist1.dae" />
+        </geometry>
+        <material name="LightGrey">
+          <color rgba="0.7 0.7 0.7 1.0"/>
+        </material>
+      </visual>
+      <collision>
+        <geometry>
+          <mesh filename="package://ur_description/meshes/ur5e/collision/wrist1.stl" />
         </geometry>
       </collision>
@@ -242,13 +242,13 @@
       <visual>
         <geometry>
-          <mesh filename="package://ur_description/meshes/ur5/visual/wrist2.dae" />
-        </geometry>
-        <material name="LightGrey">
-          <color rgba="0.7 0.7 0.7 1.0"/>
-        </material>
-      </visual>
-      <collision>
-        <geometry>
-          <mesh filename="package://ur_description/meshes/ur5/collision/wrist2.stl" />
+          <mesh filename="package://ur_description/meshes/ur5e/visual/wrist2.dae" />
+        </geometry>
+        <material name="LightGrey">
+          <color rgba="0.7 0.7 0.7 1.0"/>
+        </material>
+      </visual>
+      <collision>
+        <geometry>
+          <mesh filename="package://ur_description/meshes/ur5e/collision/wrist2.stl" />
         </geometry>
       </collision>
@@ -273,13 +273,13 @@
       <visual>
         <geometry>
-          <mesh filename="package://ur_description/meshes/ur5/visual/wrist3.dae" />
-        </geometry>
-        <material name="LightGrey">
-          <color rgba="0.7 0.7 0.7 1.0"/>
-        </material>
-      </visual>
-      <collision>
-        <geometry>
-          <mesh filename="package://ur_description/meshes/ur5/collision/wrist3.stl" />
+          <mesh filename="package://ur_description/meshes/ur5e/visual/wrist3.dae" />
+        </geometry>
+        <material name="LightGrey">
+          <color rgba="0.7 0.7 0.7 1.0"/>
+        </material>
+      </visual>
+      <collision>
+        <geometry>
+          <mesh filename="package://ur_description/meshes/ur5e/collision/wrist3.stl" />
         </geometry>
       </collision>
