Commit message: Remove wires from E-Series bases (#22)

File: ur_description/urdf/ur10e.urdf.xacro (robot description, xacro)
@@ -62,5 +62,5 @@
     <link name="${prefix}base_link" >
       <visual>
-        <origin xyz="0.0 0.0 0.0" rpy="0.0 0.0 ${rotational_offset}"/>
+        <origin xyz="0.0 0.0 0.0" rpy="${pi/2.0} 0.0 ${rotational_offset}" />
         <geometry>
           <mesh filename="package://ur_description/meshes/ur10e/visual/base.dae"/>
@@ -71,5 +71,5 @@
       </visual>
       <collision>
-        <origin xyz="0.0 0.0 0.0" rpy="0.0 0.0 ${rotational_offset}"/>
+        <origin xyz="0.0 0.0 0.0" rpy="${pi/2.0} 0.0 ${rotational_offset}" />
         <geometry>
           <mesh filename="package://ur_description/meshes/ur10e/collision/base.dae"/>

File: ur_description/urdf/ur10e_fixture.urdf.xacro (robot description, xacro)
@@ -63,5 +63,5 @@
     <link name="${prefix}base_link" >
       <visual>
-        <origin xyz="0.0 0.0 0.0" rpy="0.0 0.0 ${rotational_offset}"/>
+        <origin xyz="0.0 0.0 0.0" rpy="${pi/2.0} 0.0 ${rotational_offset}" />
         <geometry>
           <mesh filename="package://ur_description/meshes/ur10e/visual/base.dae"/>
@@ -72,5 +72,5 @@
       </visual>
       <collision>
-        <origin xyz="0.0 0.0 0.0" rpy="0.0 0.0 ${rotational_offset}"/>
+        <origin xyz="0.0 0.0 0.0" rpy="${pi/2.0} 0.0 ${rotational_offset}" />
         <geometry>
           <mesh filename="package://ur_description/meshes/ur10e/collision/base.dae"/>

File: ur_description/urdf/ur3e.urdf.xacro (robot description, xacro)
@@ -60,5 +60,5 @@
     <link name="${prefix}base_link" >
       <visual>
-        <origin xyz="0.0 0.0 0.0" rpy="0.0 0.0 ${rotational_offset}" />
+        <origin xyz="0.0 0.0 0.0" rpy="${pi/2.0} 0.0 ${rotational_offset}" />
         <geometry>
           <mesh filename="package://ur_description/meshes/ur3e/visual/base.dae"/>
@@ -69,5 +69,5 @@
       </visual>
       <collision>
-        <origin xyz="0.0 0.0 0.0" rpy="0.0 0.0 ${rotational_offset}" />
+        <origin xyz="0.0 0.0 0.0" rpy="${pi/2.0} 0.0 ${rotational_offset}" />
         <geometry>
           <mesh filename="package://ur_description/meshes/ur3e/collision/base.dae"/>

File: ur_description/urdf/ur3e_fixture.urdf.xacro (robot description, xacro)
@@ -61,5 +61,5 @@
     <link name="${prefix}base_link" >
       <visual>
-        <origin xyz="0.0 0.0 0.0" rpy="0.0 0.0 ${rotational_offset}" />
+        <origin xyz="0.0 0.0 0.0" rpy="${pi/2.0} 0.0 ${rotational_offset}" />
         <geometry>
           <mesh filename="package://ur_description/meshes/ur3e/visual/base.dae"/>
@@ -70,5 +70,5 @@
       </visual>
       <collision>
-        <origin xyz="0.0 0.0 0.0" rpy="0.0 0.0 ${rotational_offset}" />
+        <origin xyz="0.0 0.0 0.0" rpy="${pi/2.0} 0.0 ${rotational_offset}" />
         <geometry>
           <mesh filename="package://ur_description/meshes/ur3e/collision/base.dae"/>

File: ur_description/urdf/ur5e.urdf.xacro (robot description, xacro)
@@ -68,5 +68,5 @@
     <link name="${prefix}base_link" >
       <visual>
-        <origin xyz="0.0 0.0 0.0" rpy="0.0 0.0 ${rotational_offset}" />
+        <origin xyz="0.0 0.0 0.0" rpy="${pi/2.0} 0.0 ${rotational_offset}" />
         <geometry>
           <mesh filename="package://ur_description/meshes/ur5e/visual/base.dae" />
@@ -77,5 +77,5 @@
       </visual>
       <collision>
-        <origin xyz="0.0 0.0 0.0" rpy="0.0 0.0 ${rotational_offset}" />
+        <origin xyz="0.0 0.0 0.0" rpy="${pi/2.0} 0.0 ${rotational_offset}" />
         <geometry>
           <mesh filename="package://ur_description/meshes/ur5e/collision/base.dae" />

File: ur_description/urdf/ur5e_fixture.urdf.xacro (robot description, xacro)
@@ -68,5 +68,5 @@
     <link name="${prefix}base_link" >
       <visual>
-        <origin xyz="0.0 0.0 0.0" rpy="0.0 0.0 ${rotational_offset}" />
+        <origin xyz="0.0 0.0 0.0" rpy="${pi/2.0} 0.0 ${rotational_offset}" />
         <geometry>
           <mesh filename="package://ur_description/meshes/ur5e/visual/base.dae" />
@@ -77,5 +77,5 @@
       </visual>
       <collision>
-        <origin xyz="0.0 0.0 0.0" rpy="0.0 0.0 ${rotational_offset}" />
+        <origin xyz="0.0 0.0 0.0" rpy="${pi/2.0} 0.0 ${rotational_offset}" />
         <geometry>
           <mesh filename="package://ur_description/meshes/ur5e/collision/base.dae" />
