Commit message: Allow for 4 rotations of wrist3

File: ur_description/urdf/ur3e.urdf.xacro (robot description, xacro)
@@ -249,5 +249,5 @@
       <axis xyz="0 1 0" />
       <xacro:unless value="${joint_limited}">
-        <limit lower="${-2.0 * pi}" upper="${2.0 * pi}" effort="54.0" velocity="3.2"/>
+        <limit lower="${-4 * 2.0 * pi}" upper="${4 * 2.0 * pi}" effort="54.0" velocity="3.2"/>
       </xacro:unless>
       <xacro:if value="${joint_limited}">

File: ur_description/urdf/ur3e_fixture.urdf.xacro (robot description, xacro)
@@ -85,5 +85,5 @@
       <axis xyz="0 0 1" />
       <xacro:unless value="${joint_limited}">
-        <limit lower="${-large_joint_limits}" upper="${large_joint_limits}" effort="330.0" velocity="2.16"/>
+        <limit lower="${-4 * 2.0 * pi}" upper="${4 * 2.0 * pi}" effort="330.0" velocity="2.16"/>
       </xacro:unless>
       <xacro:if value="${joint_limited}">
