Commit message: [TF-4327] Epic frame redesign (#28)
* [RPI-6] Remove references to teachmate links in SRDFs (#24)

* Make base the root frame (#26)

* Removing stand frame, it's possible all of these files may be deleted

* Update fixed reference frame (#27)

* Update urdf robot names

File: ur_description/urdf/ur10.urdf.xacro (robot description, xacro)
@@ -281,6 +281,6 @@
       -->
       <origin xyz="0 0 0" rpy="0 0 ${-pi}"/>
-      <parent link="${prefix}base_link"/>
-      <child link="${prefix}base"/>
+      <parent link="${prefix}base"/>
+      <child link="${prefix}base_link"/>
     </joint>
     <!-- Frame coincident with all-zeros TCP on UR controller -->

File: ur_description/urdf/ur10_fixture.urdf.xacro (robot description, xacro)
@@ -282,6 +282,6 @@
       -->
       <origin xyz="0 0 0" rpy="0 0 ${-pi}"/>
-      <parent link="${prefix}base_link"/>
-      <child link="${prefix}base"/>
+      <parent link="${prefix}base"/>
+      <child link="${prefix}base_link"/>
     </joint>
     <!-- Frame coincident with all-zeros TCP on UR controller -->

File: ur_description/urdf/ur10_joint_limited_robot.urdf.xacro (robot description, xacro)
@@ -1,5 +1,4 @@
 <?xml version="1.0"?>
-<robot xmlns:xacro="http://www.ros.org/wiki/xacro"
-       name="ur10" >
+<robot xmlns:xacro="http://www.ros.org/wiki/xacro" name="READY_UR10" >
   <!-- common stuff -->
   <xacro:include filename="$(find ur_description)/urdf/common.gazebo.xacro" />
@@ -8,9 +7,3 @@
   <!-- arm -->
   <xacro:ur10_robot prefix="" joint_limited="true"/>
-  <link name="stand" />
-  <joint name="world_joint" type="fixed">
-    <parent link="stand" />
-    <child link = "base_link" />
-    <origin xyz="0.0 0.0 0.0" rpy="0.0 0.0 0.0" />
-  </joint>
 </robot>

File: ur_description/urdf/ur10_robot.urdf.xacro (robot description, xacro)
@@ -1,5 +1,4 @@
 <?xml version="1.0"?>
-<robot xmlns:xacro="http://www.ros.org/wiki/xacro"
-       name="ur10" >
+<robot xmlns:xacro="http://www.ros.org/wiki/xacro" name="READY_UR10" >
   <!-- common stuff -->
   <xacro:include filename="$(find ur_description)/urdf/common.gazebo.xacro" />
@@ -8,9 +7,3 @@
   <!-- arm -->
   <xacro:ur10_robot prefix="" joint_limited="false"/>
-  <link name="stand" />
-  <joint name="world_joint" type="fixed">
-    <parent link="stand" />
-    <child link = "base_link" />
-    <origin xyz="0.0 0.0 0.0" rpy="0.0 0.0 0.0" />
-  </joint>
 </robot>

File: ur_description/urdf/ur10e.urdf.xacro (robot description, xacro)
@@ -301,6 +301,6 @@
       -->
       <origin xyz="0 0 0" rpy="0 0 ${-pi}"/>
-      <parent link="${prefix}base_link"/>
-      <child link="${prefix}base"/>
+      <parent link="${prefix}base"/>
+      <child link="${prefix}base_link"/>
     </joint>
     <!-- Frame coincident with all-zeros TCP on UR controller -->

File: ur_description/urdf/ur10e_fixture.urdf.xacro (robot description, xacro)
@@ -302,6 +302,6 @@
       -->
       <origin xyz="0 0 0" rpy="0 0 ${-pi}"/>
-      <parent link="${prefix}base_link"/>
-      <child link="${prefix}base"/>
+      <parent link="${prefix}base"/>
+      <child link="${prefix}base_link"/>
     </joint>
     <!-- Frame coincident with all-zeros TCP on UR controller -->

File: ur_description/urdf/ur10e_joint_limited_robot.urdf.xacro (robot description, xacro)
@@ -1,5 +1,4 @@
 <?xml version="1.0"?>
-<robot xmlns:xacro="http://www.ros.org/wiki/xacro"
-       name="READY_UR10E" >
+<robot xmlns:xacro="http://www.ros.org/wiki/xacro" name="READY_UR10E" >
   <!-- common stuff -->
   <xacro:include filename="$(find ur_description)/urdf/common.gazebo.xacro" />
@@ -8,9 +7,3 @@
   <!-- arm -->
   <xacro:ur10_robot prefix="" joint_limited="true"/>
-  <link name="stand" />
-  <joint name="world_joint" type="fixed">
-    <parent link="stand" />
-    <child link = "base_link" />
-    <origin xyz="0.0 0.0 0.0" rpy="0.0 0.0 0.0" />
-  </joint>
 </robot>

File: ur_description/urdf/ur10e_robot.urdf.xacro (robot description, xacro)
@@ -1,5 +1,4 @@
 <?xml version="1.0"?>
-<robot xmlns:xacro="http://www.ros.org/wiki/xacro"
-       name="READY_UR10E" >
+<robot xmlns:xacro="http://www.ros.org/wiki/xacro" name="READY_UR10E" >
   <!-- common stuff -->
   <xacro:include filename="$(find ur_description)/urdf/common.gazebo.xacro" />
@@ -8,9 +7,3 @@
   <!-- arm -->
   <xacro:ur10_robot prefix="" joint_limited="false"/>
-  <link name="stand" />
-  <joint name="world_joint" type="fixed">
-    <parent link="stand" />
-    <child link = "base_link" />
-    <origin xyz="0.0 0.0 0.0" rpy="0.0 0.0 0.0" />
-  </joint>
 </robot>

File: ur_description/urdf/ur3.urdf.xacro (robot description, xacro)
@@ -280,6 +280,6 @@
       -->
       <origin xyz="0 0 0" rpy="0 0 ${-pi}"/>
-      <parent link="${prefix}base_link"/>
-      <child link="${prefix}base"/>
+      <parent link="${prefix}base"/>
+      <child link="${prefix}base_link"/>
     </joint>
     <!-- Frame coincident with all-zeros TCP on UR controller -->

File: ur_description/urdf/ur3_fixture.urdf.xacro (robot description, xacro)
@@ -281,6 +281,6 @@
       -->
       <origin xyz="0 0 0" rpy="0 0 ${-pi}"/>
-      <parent link="${prefix}base_link"/>
-      <child link="${prefix}base"/>
+      <parent link="${prefix}base"/>
+      <child link="${prefix}base_link"/>
     </joint>
     <!-- Frame coincident with all-zeros TCP on UR controller -->

File: ur_description/urdf/ur3_joint_limited_robot.urdf.xacro (robot description, xacro)
@@ -1,5 +1,4 @@
 <?xml version="1.0"?>
-<robot xmlns:xacro="http://www.ros.org/wiki/xacro"
-       name="ur3" >
+<robot xmlns:xacro="http://www.ros.org/wiki/xacro" name="READY_UR3" >
   <!-- common stuff -->
   <xacro:include filename="$(find ur_description)/urdf/common.gazebo.xacro" />
@@ -8,9 +7,3 @@
   <!-- arm -->
   <xacro:ur3_robot prefix="" joint_limited="true"/>
-  <link name="stand" />
-  <joint name="world_joint" type="fixed">
-    <parent link="stand" />
-    <child link = "base_link" />
-    <origin xyz="0.0 0.0 0.0" rpy="0.0 0.0 0.0" />
-  </joint>
 </robot>

File: ur_description/urdf/ur3_robot.urdf.xacro (robot description, xacro)
@@ -1,5 +1,4 @@
 <?xml version="1.0"?>
-<robot xmlns:xacro="http://www.ros.org/wiki/xacro"
-       name="ur3" >
+<robot xmlns:xacro="http://www.ros.org/wiki/xacro" name="READY_UR3" >
   <!-- common stuff -->
   <xacro:include filename="$(find ur_description)/urdf/common.gazebo.xacro" />
@@ -8,9 +7,3 @@
   <!-- arm -->
   <xacro:ur3_robot prefix="" joint_limited="false"/>
-  <link name="stand" />
-  <joint name="world_joint" type="fixed">
-    <parent link="stand" />
-    <child link = "base_link" />
-    <origin xyz="0.0 0.0 0.0" rpy="0.0 0.0 0.0" />
-  </joint>
 </robot>

File: ur_description/urdf/ur3e.urdf.xacro (robot description, xacro)
@@ -299,6 +299,6 @@
       -->
       <origin xyz="0 0 0" rpy="0 0 ${-pi}"/>
-      <parent link="${prefix}base_link"/>
-      <child link="${prefix}base"/>
+      <parent link="${prefix}base"/>
+      <child link="${prefix}base_link"/>
     </joint>
     <!-- Frame coincident with all-zeros TCP on UR controller -->

File: ur_description/urdf/ur3e_fixture.urdf.xacro (robot description, xacro)
@@ -300,6 +300,6 @@
       -->
       <origin xyz="0 0 0" rpy="0 0 ${-pi}"/>
-      <parent link="${prefix}base_link"/>
-      <child link="${prefix}base"/>
+      <parent link="${prefix}base"/>
+      <child link="${prefix}base_link"/>
     </joint>
     <!-- Frame coincident with all-zeros TCP on UR controller -->

File: ur_description/urdf/ur3e_joint_limited_robot.urdf.xacro (robot description, xacro)
@@ -1,5 +1,4 @@
 <?xml version="1.0"?>
-<robot xmlns:xacro="http://www.ros.org/wiki/xacro"
-       name="READY_UR3E" >
+<robot xmlns:xacro="http://www.ros.org/wiki/xacro" name="READY_UR3E" >
   <!-- common stuff -->
   <xacro:include filename="$(find ur_description)/urdf/common.gazebo.xacro" />
@@ -8,9 +7,3 @@
   <!-- arm -->
   <xacro:ur3_robot prefix="" joint_limited="true"/>
-  <link name="stand" />
-  <joint name="world_joint" type="fixed">
-    <parent link="stand" />
-    <child link = "base_link" />
-    <origin xyz="0.0 0.0 0.0" rpy="0.0 0.0 0.0" />
-  </joint>
 </robot>

File: ur_description/urdf/ur3e_robot.urdf.xacro (robot description, xacro)
@@ -1,5 +1,4 @@
 <?xml version="1.0"?>
-<robot xmlns:xacro="http://www.ros.org/wiki/xacro"
-       name="READY_UR3E" >
+<robot xmlns:xacro="http://www.ros.org/wiki/xacro" name="READY_UR3E" >
   <!-- common stuff -->
   <xacro:include filename="$(find ur_description)/urdf/common.gazebo.xacro" />
@@ -8,9 +7,3 @@
   <!-- arm -->
   <xacro:ur3_robot prefix="" joint_limited="false"/>
-  <link name="stand" />
-  <joint name="world_joint" type="fixed">
-    <parent link="stand" />
-    <child link = "base_link" />
-    <origin xyz="0.0 0.0 0.0" rpy="0.0 0.0 0.0" />
-  </joint>
 </robot>

File: ur_description/urdf/ur5.urdf.xacro (robot description, xacro)
@@ -296,6 +296,6 @@
       -->
       <origin xyz="0 0 0" rpy="0 0 ${-pi}"/>
-      <parent link="${prefix}base_link"/>
-      <child link="${prefix}base"/>
+      <parent link="${prefix}base"/>
+      <child link="${prefix}base_link"/>
     </joint>
     <!-- Frame coincident with all-zeros TCP on UR controller -->

File: ur_description/urdf/ur5_fixture.urdf.xacro (robot description, xacro)
@@ -388,7 +388,7 @@
                  not corrected wrt the real robot (ie: rotated over 180
                  degrees)-->
-        <origin xyz="0 0 0" rpy="0 0 ${-pi}"/>
-        <parent link="${prefix}base_link"/>
-        <child link="${prefix}base"/>
+        <origin xyz="0 0 0" rpy="0 0 -${pi}"/>
+        <parent link="${prefix}base"/>
+        <child link="${prefix}base_link"/>
     </joint>
     <!-- Frame coincident with all-zeros TCP on UR controller -->

File: ur_description/urdf/ur5_joint_limited_robot.urdf.xacro (robot description, xacro)
@@ -1,5 +1,4 @@
 <?xml version="1.0"?>
-<robot xmlns:xacro="http://www.ros.org/wiki/xacro"
-       name="READY_UR5" >
+<robot xmlns:xacro="http://www.ros.org/wiki/xacro" name="READY_UR5" >
   <!-- common stuff -->
   <xacro:include filename="$(find ur_description)/urdf/common.gazebo.xacro" />
@@ -8,9 +7,3 @@
   <!-- arm -->
   <xacro:ur5_robot prefix="" joint_limited="true"/>
-  <link name="stand" />
-  <joint name="world_joint" type="fixed">
-    <parent link="stand" />
-    <child link = "base_link" />
-    <origin xyz="0.0 0.0 0.0" rpy="0.0 0.0 0.0" />
-  </joint>
 </robot>

File: ur_description/urdf/ur5_robot.urdf.xacro (robot description, xacro)
@@ -1,5 +1,4 @@
 <?xml version="1.0"?>
-<robot xmlns:xacro="http://www.ros.org/wiki/xacro"
-       name="READY_UR5" >
+<robot xmlns:xacro="http://www.ros.org/wiki/xacro" name="READY_UR5" >
   <!-- common stuff -->
   <xacro:include filename="$(find ur_description)/urdf/common.gazebo.xacro" />
@@ -8,9 +7,3 @@
   <!-- arm -->
   <xacro:ur5_robot prefix="" joint_limited="false"/>
-  <link name="stand" />
-  <joint name="world_joint" type="fixed">
-    <parent link="stand" />
-    <child link = "base_link" />
-    <origin xyz="0.0 0.0 0.0" rpy="0.0 0.0 0.0" />
-  </joint>
 </robot>
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